File: Eagle/Word-Clock.brd (EAGLE design)
At the start: 280 x 280 mm, 191 parts, among them IC1 7805T, IC2 LM2936Z-3.3, IC3 UDN2981A, IC4 UDN2981A, IC5 DS3231/SO, IC6 LM358N, J1 USB-MINIB-5PIN, J4 3x2M, Q1 BS250, Q3 16MHz, U1 TLC5940-NT, U2 TLC5940-NT, U3 TLC5940-NT

Commit message: Schematic & PCB V1.2
Parts:
- removed IC1: 7805T, linear:TO220H
- removed IC6: LM358N, linear:DIL08
- removed J1: USB-MINIB-5PIN, SparkFun-Connectors:USB-MINIB
- removed J4: 3x2M, pinhead:2X03/90
- removed JP1: POWER_JACKPTH, SparkFun-Connectors:POWER_JACK_PTH
- removed L2: MH2029-300Y, resistor:0207/7
- removed Q3: 16MHz, crystal:HC49U-V
- removed R12: 2.2K, resistor:0207/7
- removed R13, R14: 10K, resistor:0207/7
- removed U$4: ATMEGA32U4-AU, adafruit:TQFP44
- removed U2, U3: TLC5940-NT, SparkFun-DigitalIC:DIL28-3
- added C15: 22pF, resistor:C050-024X044
- added D3, D4: (no value), SparkFun-LED:LED-1206
- added I1: (no value), rcl:0207/7
- added JP2: USBPTH-VERTICAL, SparkFun-Connectors:USB-B-PTH-VERTICAL
- added JP3: (no value), SparkFun-Connectors:2X3-SHROUDED
- added JP4: (no value), SparkFun-Connectors:MOLEX-1X2
- added R2, R9: 10k, resistor:0207/7
- added S2, S3, S4: SWITCH-MOMENTARY-2SIDE_EZ, SparkFun-Electromechanical:TACTILE-PTH-SIDEEZ
- added Y1: 16MHz, SparkFun-FreqCtrl:HC49U-V
- C1, C3: value 22u -> 100uF
- C10, C2, C8, C9: value 100n -> 100nF; device resistor:C050-025X075 -> capacitor-wima:C5B2.5
- C11: value 100n -> 1uF; device resistor:C050-025X075 -> resistor:E2,5-6
- C12: value 22pF -> 100nF; device resistor:C050-024X044 -> capacitor-wima:C5B2.5
- C13: value 22pF -> 1uF; device resistor:C050-024X044 -> resistor:E2,5-6
- C14: value 22u -> 22pF; device resistor:E2,5-6 -> resistor:C050-024X044
- C4, C6: value 1uF -> 100nF; device resistor:E2,5-6 -> capacitor-wima:C5B2.5
- C5: value 100n -> 100uF; device resistor:C050-025X075 -> resistor:E2,5-6
- C7: device resistor:C050-025X075 -> capacitor-wima:C5B2.5
- D1: value 1N4148DO35-10 -> 1N4001; device diode:DO35-10 -> diode:DO41-10
- D2: value 1N5817-B -> 1N4148; device diode:DO41-7.6 -> diode:DO35-7
- F1: value MF-MSMF050-2 500mA -> 500mA; device rcl:L1812 -> adafruit:R1206
- IC3: value UDN2981A -> LM358N; device uln-udn:DIL18 -> linear:DIL08
- IC4: value UDN2981A -> DS3231/SO; device uln-udn:DIL18 -> adafruit:SO16W
- IC5: value DS3231/SO -> LM340H-05; device adafruit:SO16W -> linear:TO220H
- LED1, LED10, LED100, LED101, LED102, LED103, LED104, LED105, LED106, LED107, LED108, LED109, LED11, LED110, LED111, LED112, LED113, LED114, LED115, LED116, LED117, LED118, LED119, LED12, LED120, LED121, LED122, LED123, LED124, LED125, LED126, LED127, LED128, LED129, LED13, LED130, LED131, LED132, LED133, LED134, LED135, LED136, LED137, LED138, LED139, LED14, LED140, LED141, LED142, LED143, LED144, LED15, LED16, LED17, LED18, LED19, LED2, LED20, LED21, LED22, LED23, LED24, LED25, LED26, LED27, LED28, LED29, LED3, LED30, LED31, LED32, LED33, LED34, LED35, LED36, LED37, LED38, LED39, LED4, LED40, LED41, LED42, LED43, LED44, LED45, LED46, LED47, LED48, LED49, LED5, LED50, LED51, LED52, LED53, LED54, LED55, LED56, LED57, LED58, LED59, LED6, LED60, LED61, LED62, LED63, LED64, LED65, LED66, LED67, LED68, LED69, LED7, LED70, LED71, LED72, LED73, LED74, LED75, LED76, LED77, LED78, LED79, LED8, LED80, LED81, LED82, LED83, LED84, LED85, LED86, LED87, LED88, LED89, LED9, LED90, LED91, LED92, LED93, LED94, LED95, LED96, LED97, LED98, LED99: value RGBLED5050 -> WS2812B; device adafruit:RGBLED5050 -> adafruit:WS2812B
- Q1: value BS250 -> PFETBS250; device transistor-small-signal:SOT54E -> adafruit:TO92-OVAL
- R1: value 10K -> 10k
- R10, R11: value 2.2K -> 1K
- R3: value 22R -> 10k
- R4: value 22R -> PHOTOCELLPTH; device resistor:0207/7 -> SparkFun-Sensors:PHOTOCELL
- R5: value 2.2K -> 10k
- R6: value 10K -> 22R
- R7: value 2.2K -> 22R
- R8: value 2.2K -> 1M
- S1: value SWITCH-MOMENTARY-212MM -> (none); device SparkFun-Electromechanical:TACTILE-PTH-12MM -> SparkFun-Electromechanical:TACTILE-PTH
- U1: value TLC5940-NT -> ATMEGA32U4TQFP-44; device SparkFun-DigitalIC:DIL28-3 -> SparkFun-DigitalIC:TQFP44
- moved R6 332.1 mm to (129.0, 20.0), flipped to the bottom
- moved C14 316.2 mm to (140.0, 4.00), flipped to the bottom
- moved R3 312.4 mm to (128.0, 6.00), flipped to the bottom, turned to 270 degrees
- moved R4 308.7 mm to (145.9, 68.4), flipped to the bottom, turned to 180 degrees
- moved R5 303.3 mm to (102.0, 14.0), flipped to the bottom, turned to 180 degrees
- moved C11 297.5 mm to (141.0, 23.0), flipped to the bottom, turned to 180 degrees
- moved C1 291.6 mm to (80.0, 4.00), flipped to the bottom, turned to 180 degrees
- moved S1 283.2 mm to (176.5, 5.00), flipped to the bottom
- moved C6 282.0 mm to (84.0, 12.0), flipped to the bottom, turned to 270 degrees
- moved C4 271.2 mm to (81.0, 12.0), flipped to the bottom, turned to 90 degrees
- moved IC2 267.4 mm to (102.0, 4.00), flipped to the bottom, turned to 180 degrees
- moved C8 263.0 mm to (111.0, 2.00), flipped to the bottom, turned to 180 degrees
- moved C7 262.3 mm to (119.0, 2.00), flipped to the bottom
- moved C10 260.6 mm to (102.0, 17.0), flipped to the bottom
- moved U1 258.9 mm to (115.0, 12.0), flipped to the bottom, turned to 315 degrees
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Connections:
- removed net +5V: C10.1, C11.1, C2.1, C3.+, D1.C, IC1.3, IC2.3, IC5.2, IC6.8, J4.2, L2.1, Q1.S, R1.1, U$4.14, U$4.2, U$4.24, U$4.34
- removed net 3V3: C4.+, IC2.1, IC6.2
- removed net A0: IC4.4, U$4.36
- removed net A1: IC4.5, U$4.37
- removed net A2: IC4.6, U$4.38
- removed net A3: U$4.39
- removed net A4: U$4.40
- removed net A5: U$4.41
- removed net AVCC1: C7.1, L2.2, U$4.44
- removed net C10BLUE: LED10.4, LED106.4, LED118.4, LED130.4, LED142.4, LED22.4, LED34.4, LED46.4, LED58.4, LED70.4, LED82.4, LED94.4, U3.6
- removed net C10GRN: LED10.6, LED106.6, LED118.6, LED130.6, LED142.6, LED22.6, LED34.6, LED46.6, LED58.6, LED70.6, LED82.6, LED94.6, U3.4
- removed net C10RED: LED10.5, LED106.5, LED118.5, LED130.5, LED142.5, LED22.5, LED34.5, LED46.5, LED58.5, LED70.5, LED82.5, LED94.5, U3.5
- removed net C11BLUE: LED107.4, LED11.4, LED119.4, LED131.4, LED143.4, LED23.4, LED35.4, LED47.4, LED59.4, LED71.4, LED83.4, LED95.4, U3.9
- removed net C11GRN: LED107.6, LED11.6, LED119.6, LED131.6, LED143.6, LED23.6, LED35.6, LED47.6, LED59.6, LED71.6, LED83.6, LED95.6, U3.7
- removed net C11RED: LED107.5, LED11.5, LED119.5, LED131.5, LED143.5, LED23.5, LED35.5, LED47.5, LED59.5, LED71.5, LED83.5, LED95.5, U3.8
- removed net C12BLUE: LED108.4, LED12.4, LED120.4, LED132.4, LED144.4, LED24.4, LED36.4, LED48.4, LED60.4, LED72.4, LED84.4, LED96.4, U3.12
- removed net C12GRN: LED108.6, LED12.6, LED120.6, LED132.6, LED144.6, LED24.6, LED36.6, LED48.6, LED60.6, LED72.6, LED84.6, LED96.6, U3.10
- removed net C12RED: LED108.5, LED12.5, LED120.5, LED132.5, LED144.5, LED24.5, LED36.5, LED48.5, LED60.5, LED72.5, LED84.5, LED96.5, U3.11
- removed net C1BLUE: LED1.4, LED109.4, LED121.4, LED13.4, LED133.4, LED25.4, LED37.4, LED49.4, LED61.4, LED73.4, LED85.4, LED97.4, U1.3
- removed net C1GRN: LED1.6, LED109.6, LED121.6, LED13.6, LED133.6, LED25.6, LED37.6, LED49.6, LED61.6, LED73.6, LED85.6, LED97.6, U1.1
- removed net C1RED: LED1.5, LED109.5, LED121.5, LED13.5, LED133.5, LED25.5, LED37.5, LED49.5, LED61.5, LED73.5, LED85.5, LED97.5, U1.2
- removed net C2BLUE: LED110.4, LED122.4, LED134.4, LED14.4, LED2.4, LED26.4, LED38.4, LED50.4, LED62.4, LED74.4, LED86.4, LED98.4, U1.6
- removed net C2GRN: LED110.6, LED122.6, LED134.6, LED14.6, LED2.6, LED26.6, LED38.6, LED50.6, LED62.6, LED74.6, LED86.6, LED98.6, U1.4
- removed net C2RED: LED110.5, LED122.5, LED134.5, LED14.5, LED2.5, LED26.5, LED38.5, LED50.5, LED62.5, LED74.5, LED86.5, LED98.5, U1.5
- removed net C3BLUE: LED111.4, LED123.4, LED135.4, LED15.4, LED27.4, LED3.4, LED39.4, LED51.4, LED63.4, LED75.4, LED87.4, LED99.4, U1.9
- removed net C3GRN: LED111.6, LED123.6, LED135.6, LED15.6, LED27.6, LED3.6, LED39.6, LED51.6, LED63.6, LED75.6, LED87.6, LED99.6, U1.7
- removed net C3RED: LED111.5, LED123.5, LED135.5, LED15.5, LED27.5, LED3.5, LED39.5, LED51.5, LED63.5, LED75.5, LED87.5, LED99.5, U1.8
- removed net C4BLUE: LED100.4, LED112.4, LED124.4, LED136.4, LED16.4, LED28.4, LED4.4, LED40.4, LED52.4, LED64.4, LED76.4, LED88.4, U1.12
- removed net C4GRN: LED100.6, LED112.6, LED124.6, LED136.6, LED16.6, LED28.6, LED4.6, LED40.6, LED52.6, LED64.6, LED76.6, LED88.6, U1.10
- removed net C4RED: LED100.5, LED112.5, LED124.5, LED136.5, LED16.5, LED28.5, LED4.5, LED40.5, LED52.5, LED64.5, LED76.5, LED88.5, U1.11
- removed net C5BLUE: LED101.4, LED113.4, LED125.4, LED137.4, LED17.4, LED29.4, LED41.4, LED5.4, LED53.4, LED65.4, LED77.4, LED89.4, U2.3
- removed net C5GRN: LED101.6, LED113.6, LED125.6, LED137.6, LED17.6, LED29.6, LED41.6, LED5.6, LED53.6, LED65.6, LED77.6, LED89.6, U2.1
- removed net C5RED: LED101.5, LED113.5, LED125.5, LED137.5, LED17.5, LED29.5, LED41.5, LED5.5, LED53.5, LED65.5, LED77.5, LED89.5, U2.2
- removed net C6BLUE: LED102.4, LED114.4, LED126.4, LED138.4, LED18.4, LED30.4, LED42.4, LED54.4, LED6.4, LED66.4, LED78.4, LED90.4, U2.6
- removed net C6GRN: LED102.6, LED114.6, LED126.6, LED138.6, LED18.6, LED30.6, LED42.6, LED54.6, LED6.6, LED66.6, LED78.6, LED90.6, U2.4
- removed net C6RED: LED102.5, LED114.5, LED126.5, LED138.5, LED18.5, LED30.5, LED42.5, LED54.5, LED6.5, LED66.5, LED78.5, LED90.5, U2.5
- removed net C7BLUE: LED103.4, LED115.4, LED127.4, LED139.4, LED19.4, LED31.4, LED43.4, LED55.4, LED67.4, LED7.4, LED79.4, LED91.4, U2.9
- removed net C7GRN: LED103.6, LED115.6, LED127.6, LED139.6, LED19.6, LED31.6, LED43.6, LED55.6, LED67.6, LED7.6, LED79.6, LED91.6, U2.7
- removed net C7RED: LED103.5, LED115.5, LED127.5, LED139.5, LED19.5, LED31.5, LED43.5, LED55.5, LED67.5, LED7.5, LED79.5, LED91.5, U2.8
- removed net C8BLUE: LED104.4, LED116.4, LED128.4, LED140.4, LED20.4, LED32.4, LED44.4, LED56.4, LED68.4, LED8.4, LED80.4, LED92.4, U2.12
- removed net C8GRN: LED104.6, LED116.6, LED128.6, LED140.6, LED20.6, LED32.6, LED44.6, LED56.6, LED68.6, LED8.6, LED80.6, LED92.6, U2.10
- removed net C8RED: LED104.5, LED116.5, LED128.5, LED140.5, LED20.5, LED32.5, LED44.5, LED56.5, LED68.5, LED8.5, LED80.5, LED92.5, U2.11
- removed net C9BLUE: LED105.4, LED117.4, LED129.4, LED141.4, LED21.4, LED33.4, LED45.4, LED57.4, LED69.4, LED81.4, LED9.4, LED93.4, U3.3
- removed net C9GRN: LED105.6, LED117.6, LED129.6, LED141.6, LED21.6, LED33.6, LED45.6, LED57.6, LED69.6, LED81.6, LED9.6, LED93.6, U3.1
- removed net C9RED: LED105.5, LED117.5, LED129.5, LED141.5, LED21.5, LED33.5, LED45.5, LED57.5, LED69.5, LED81.5, LED9.5, LED93.5, U3.2
- removed net CMP: C8.2, IC6.3, R13.1, R14.2
- removed net D0/RX: IC3.1, U$4.20
- removed net D1/TX: IC3.2, U$4.21
- removed net D2/SDA: IC5.15, U$4.19
- removed net D3/SCL: IC5.16, U$4.18
- removed net D4*: IC3.3, U$4.25
- removed net D5*: U$4.31, U1.18, U2.18, U3.18
- removed net D6*: IC3.4, U$4.27
- removed net D7: IC3.5, U$4.1
- removed net IO10*: R10.2, R11.2, R12.2, U$4.30, U1.23, U2.23, U3.23
- removed net IO11*: IC4.1, U$4.12
- removed net IO12*: IC4.2, U$4.26
- removed net IO13*: IC4.3, U$4.32
- removed net IO8: IC3.6, U$4.28
- removed net IO9*: U$4.29, U1.24, U2.24, U3.24
- removed net R1: IC3.18, LED1.1, LED1.2, LED1.3, LED10.1, LED10.2, LED10.3, LED11.1, LED11.2, LED11.3, LED12.1, LED12.2, LED12.3, LED2.1, LED2.2, LED2.3, LED3.1, LED3.2, LED3.3, LED4.1, LED4.2, LED4.3, LED5.1, LED5.2, LED5.3, LED6.1, LED6.2, LED6.3, LED7.1, LED7.2, LED7.3, LED8.1, LED8.2, LED8.3, LED9.1, LED9.2, LED9.3
- removed net R10: IC4.15, LED109.1, LED109.2, LED109.3, LED110.1, LED110.2, LED110.3, LED111.1, LED111.2, LED111.3, LED112.1, LED112.2, LED112.3, LED113.1, LED113.2, LED113.3, LED114.1, LED114.2, LED114.3, LED115.1, LED115.2, LED115.3, LED116.1, LED116.2, LED116.3, LED117.1, LED117.2, LED117.3, LED118.1, LED118.2, LED118.3, LED119.1, LED119.2, LED119.3, LED120.1, LED120.2, LED120.3
- removed net R11: IC4.14, LED121.1, LED121.2, LED121.3, LED122.1, LED122.2, LED122.3, LED123.1, LED123.2, LED123.3, LED124.1, LED124.2, LED124.3, LED125.1, LED125.2, LED125.3, LED126.1, LED126.2, LED126.3, LED127.1, LED127.2, LED127.3, LED128.1, LED128.2, LED128.3, LED129.1, LED129.2, LED129.3, LED130.1, LED130.2, LED130.3, LED131.1, LED131.2, LED131.3, LED132.1, LED132.2, LED132.3
- removed net R12: IC4.13, LED133.1, LED133.2, LED133.3, LED134.1, LED134.2, LED134.3, LED135.1, LED135.2, LED135.3, LED136.1, LED136.2, LED136.3, LED137.1, LED137.2, LED137.3, LED138.1, LED138.2, LED138.3, LED139.1, LED139.2, LED139.3, LED140.1, LED140.2, LED140.3, LED141.1, LED141.2, LED141.3, LED142.1, LED142.2, LED142.3, LED143.1, LED143.2, LED143.3, LED144.1, LED144.2, LED144.3
- removed net R2: IC3.17, LED13.1, LED13.2, LED13.3, LED14.1, LED14.2, LED14.3, LED15.1, LED15.2, LED15.3, LED16.1, LED16.2, LED16.3, LED17.1, LED17.2, LED17.3, LED18.1, LED18.2, LED18.3, LED19.1, LED19.2, LED19.3, LED20.1, LED20.2, LED20.3, LED21.1, LED21.2, LED21.3, LED22.1, LED22.2, LED22.3, LED23.1, LED23.2, LED23.3, LED24.1, LED24.2, LED24.3
- removed net R3: IC3.16, LED25.1, LED25.2, LED25.3, LED26.1, LED26.2, LED26.3, LED27.1, LED27.2, LED27.3, LED28.1, LED28.2, LED28.3, LED29.1, LED29.2, LED29.3, LED30.1, LED30.2, LED30.3, LED31.1, LED31.2, LED31.3, LED32.1, LED32.2, LED32.3, LED33.1, LED33.2, LED33.3, LED34.1, LED34.2, LED34.3, LED35.1, LED35.2, LED35.3, LED36.1, LED36.2, LED36.3
- removed net R4: IC3.15, LED37.1, LED37.2, LED37.3, LED38.1, LED38.2, LED38.3, LED39.1, LED39.2, LED39.3, LED40.1, LED40.2, LED40.3, LED41.1, LED41.2, LED41.3, LED42.1, LED42.2, LED42.3, LED43.1, LED43.2, LED43.3, LED44.1, LED44.2, LED44.3, LED45.1, LED45.2, LED45.3, LED46.1, LED46.2, LED46.3, LED47.1, LED47.2, LED47.3, LED48.1, LED48.2, LED48.3
- removed net R5: IC3.14, LED49.1, LED49.2, LED49.3, LED50.1, LED50.2, LED50.3, LED51.1, LED51.2, LED51.3, LED52.1, LED52.2, LED52.3, LED53.1, LED53.2, LED53.3, LED54.1, LED54.2, LED54.3, LED55.1, LED55.2, LED55.3, LED56.1, LED56.2, LED56.3, LED57.1, LED57.2, LED57.3, LED58.1, LED58.2, LED58.3, LED59.1, LED59.2, LED59.3, LED60.1, LED60.2, LED60.3
- removed net R6: IC3.13, LED61.1, LED61.2, LED61.3, LED62.1, LED62.2, LED62.3, LED63.1, LED63.2, LED63.3, LED64.1, LED64.2, LED64.3, LED65.1, LED65.2, LED65.3, LED66.1, LED66.2, LED66.3, LED67.1, LED67.2, LED67.3, LED68.1, LED68.2, LED68.3, LED69.1, LED69.2, LED69.3, LED70.1, LED70.2, LED70.3, LED71.1, LED71.2, LED71.3, LED72.1, LED72.2, LED72.3
- removed net R7: IC4.18, LED73.1, LED73.2, LED73.3, LED74.1, LED74.2, LED74.3, LED75.1, LED75.2, LED75.3, LED76.1, LED76.2, LED76.3, LED77.1, LED77.2, LED77.3, LED78.1, LED78.2, LED78.3, LED79.1, LED79.2, LED79.3, LED80.1, LED80.2, LED80.3, LED81.1, LED81.2, LED81.3, LED82.1, LED82.2, LED82.3, LED83.1, LED83.2, LED83.3, LED84.1, LED84.2, LED84.3
- removed net R8: IC4.17, LED85.1, LED85.2, LED85.3, LED86.1, LED86.2, LED86.3, LED87.1, LED87.2, LED87.3, LED88.1, LED88.2, LED88.3, LED89.1, LED89.2, LED89.3, LED90.1, LED90.2, LED90.3, LED91.1, LED91.2, LED91.3, LED92.1, LED92.2, LED92.3, LED93.1, LED93.2, LED93.3, LED94.1, LED94.2, LED94.3, LED95.1, LED95.2, LED95.3, LED96.1, LED96.2, LED96.3
- removed net R9: IC4.16, LED100.1, LED100.2, LED100.3, LED101.1, LED101.2, LED101.3, LED102.1, LED102.2, LED102.3, LED103.1, LED103.2, LED103.3, LED104.1, LED104.2, LED104.3, LED105.1, LED105.2, LED105.3, LED106.1, LED106.2, LED106.3, LED107.1, LED107.2, LED107.3, LED108.1, LED108.2, LED108.3, LED97.1, LED97.2, LED97.3, LED98.1, LED98.2, LED98.3, LED99.1, LED99.2, LED99.3
- removed net RD+: R3.1, U$4.4
- removed net RD-: R4.1, U$4.3
- removed net RXLED/SS: U$4.8
- removed net U1>>U2: U1.17, U2.26
- removed net U2>>U3: U2.17, U3.26
- removed net UCAP: C6.+, U$4.6
- removed net VUSBD: F1.1, J1.VBUS
- removed net XTAL1: C12.2, Q3.2, U$4.17
- removed net XTAL2: C13.2, Q3.1, U$4.16
- new net 3.3V: C4.1, C5.+, IC2.1, IC3.2
- new net 5V: C2.1, C3.+, C7.1, C8.1, D2.C, I1.1, IC2.3, IC3.8, IC4.2, IC5.3, JP3.2, Q1.3, R3.2, R4.1, U1.14, U1.2, U1.24, U1.34
- new net AVCC: C9.1, I1.2, U1.44
- new net N$10: LED3.2-DOUT, LED4.4-DIN
- new net N$100: LED87.2-DOUT, LED88.4-DIN
- new net N$101: LED88.2-DOUT, LED89.4-DIN
- new net N$102: LED89.2-DOUT, LED90.4-DIN
- new net N$103: LED90.2-DOUT, LED91.4-DIN
- new net N$104: LED91.2-DOUT, LED92.4-DIN
- new net N$105: LED92.2-DOUT, LED93.4-DIN
- new net N$106: LED93.2-DOUT, LED94.4-DIN
- new net N$107: LED94.2-DOUT, LED95.4-DIN
- new net N$108: LED95.2-DOUT, LED96.4-DIN
- new net N$109: LED96.2-DOUT, LED97.4-DIN
- new net N$11: LED4.2-DOUT, LED5.4-DIN
- new net N$111: LED97.2-DOUT, LED98.4-DIN
- new net N$112: LED98.2-DOUT, LED99.4-DIN
- new net N$113: LED100.4-DIN, LED99.2-DOUT
- new net N$114: LED100.2-DOUT, LED101.4-DIN
- new net N$115: LED101.2-DOUT, LED102.4-DIN
- new net N$116: LED102.2-DOUT, LED103.4-DIN
- new net N$117: LED103.2-DOUT, LED104.4-DIN
- new net N$118: LED104.2-DOUT, LED105.4-DIN
- new net N$119: LED105.2-DOUT, LED106.4-DIN
- new net N$12: LED5.2-DOUT, LED6.4-DIN
- new net N$120: LED106.2-DOUT, LED107.4-DIN
- new net N$121: LED107.2-DOUT, LED108.4-DIN
- new net N$122: LED108.2-DOUT, LED109.4-DIN
- new net N$124: LED109.2-DOUT, LED110.4-DIN
- new net N$125: LED110.2-DOUT, LED111.4-DIN
- new net N$126: LED111.2-DOUT, LED112.4-DIN
- new net N$127: LED112.2-DOUT, LED113.4-DIN
- new net N$128: LED113.2-DOUT, LED114.4-DIN
- new net N$129: LED114.2-DOUT, LED115.4-DIN
- new net N$13: LED6.2-DOUT, LED7.4-DIN
- new net N$130: LED115.2-DOUT, LED116.4-DIN
- new net N$131: LED116.2-DOUT, LED117.4-DIN
- new net N$132: LED117.2-DOUT, LED118.4-DIN
- new net N$133: LED118.2-DOUT, LED119.4-DIN
- new net N$134: LED119.2-DOUT, LED120.4-DIN
- new net N$135: LED120.2-DOUT, LED121.4-DIN
- new net N$137: LED121.2-DOUT, LED122.4-DIN
- new net N$138: LED122.2-DOUT, LED123.4-DIN
- new net N$139: LED123.2-DOUT, LED124.4-DIN
- new net N$14: LED7.2-DOUT, LED8.4-DIN
- new net N$140: LED124.2-DOUT, LED125.4-DIN
- new net N$141: LED125.2-DOUT, LED126.4-DIN
- new net N$142: LED126.2-DOUT, LED127.4-DIN
- new net N$143: LED127.2-DOUT, LED128.4-DIN
- new net N$144: LED128.2-DOUT, LED129.4-DIN
- new net N$145: LED129.2-DOUT, LED130.4-DIN
- new net N$146: LED130.2-DOUT, LED131.4-DIN
- new net N$147: LED131.2-DOUT, LED132.4-DIN
- new net N$148: LED132.2-DOUT, LED133.4-DIN
- new net N$15: LED8.2-DOUT, LED9.4-DIN
- new net N$150: LED133.2-DOUT, LED134.4-DIN
- new net N$151: LED134.2-DOUT, LED135.4-DIN
- new net N$152: LED135.2-DOUT, LED136.4-DIN
- new net N$153: LED136.2-DOUT, LED137.4-DIN
- new net N$154: LED137.2-DOUT, LED138.4-DIN
- new net N$155: LED138.2-DOUT, LED139.4-DIN
- new net N$156: LED139.2-DOUT, LED140.4-DIN
- new net N$157: LED140.2-DOUT, LED141.4-DIN
- new net N$158: LED141.2-DOUT, LED142.4-DIN
- new net N$159: LED142.2-DOUT, LED143.4-DIN
- new net N$16: LED10.4-DIN, LED9.2-DOUT
- new net N$160: LED143.2-DOUT, LED144.4-DIN
- new net N$17: LED10.2-DOUT, LED11.4-DIN
- new net N$18: LED11.2-DOUT, LED12.4-DIN
- new net N$19: LED12.2-DOUT, LED13.4-DIN
- new net N$20: LED13.2-DOUT, LED14.4-DIN
- new net N$21: LED14.2-DOUT, LED15.4-DIN
- new net N$22: LED15.2-DOUT, LED16.4-DIN
- new net N$23: LED16.2-DOUT, LED17.4-DIN
- new net N$24: LED17.2-DOUT, LED18.4-DIN
- new net N$25: LED18.2-DOUT, LED19.4-DIN
- new net N$26: LED19.2-DOUT, LED20.4-DIN
- new net N$27: LED20.2-DOUT, LED21.4-DIN
- new net N$28: LED21.2-DOUT, LED22.4-DIN
- new net N$29: LED22.2-DOUT, LED23.4-DIN
- new net N$30: LED23.2-DOUT, LED24.4-DIN
- new net N$31: LED24.2-DOUT, LED25.4-DIN
- new net N$33: LED25.2-DOUT, LED26.4-DIN
- new net N$34: LED26.2-DOUT, LED27.4-DIN
- new net N$35: LED27.2-DOUT, LED28.4-DIN
- new net N$36: LED28.2-DOUT, LED29.4-DIN
- new net N$37: LED29.2-DOUT, LED30.4-DIN
- new net N$38: LED30.2-DOUT, LED31.4-DIN
- new net N$39: LED31.2-DOUT, LED32.4-DIN
- new net N$40: LED32.2-DOUT, LED33.4-DIN
- new net N$41: LED33.2-DOUT, LED34.4-DIN
- new net N$42: LED34.2-DOUT, LED35.4-DIN
- new net N$43: LED35.2-DOUT, LED36.4-DIN
- new net N$44: LED36.2-DOUT, LED37.4-DIN
- new net N$46: LED37.2-DOUT, LED38.4-DIN
- new net N$47: LED38.2-DOUT, LED39.4-DIN
- new net N$48: LED39.2-DOUT, LED40.4-DIN
- new net N$49: LED40.2-DOUT, LED41.4-DIN
- new net N$5: LED2.2-DOUT, LED3.4-DIN
- new net N$50: LED41.2-DOUT, LED42.4-DIN
- new net N$51: LED42.2-DOUT, LED43.4-DIN
- new net N$52: LED43.2-DOUT, LED44.4-DIN
- new net N$53: LED44.2-DOUT, LED45.4-DIN
- new net N$54: LED45.2-DOUT, LED46.4-DIN
- new net N$55: LED46.2-DOUT, LED47.4-DIN
- new net N$56: LED47.2-DOUT, LED48.4-DIN
- new net N$57: LED48.2-DOUT, LED49.4-DIN
- new net N$59: LED49.2-DOUT, LED50.4-DIN
- new net N$6: D3.A, R10.1
- new net N$60: LED50.2-DOUT, LED51.4-DIN
- new net N$61: LED51.2-DOUT, LED52.4-DIN
- new net N$62: LED52.2-DOUT, LED53.4-DIN
- new net N$63: LED53.2-DOUT, LED54.4-DIN
- new net N$64: LED54.2-DOUT, LED55.4-DIN
- new net N$65: LED55.2-DOUT, LED56.4-DIN
- new net N$66: LED56.2-DOUT, LED57.4-DIN
- new net N$67: LED57.2-DOUT, LED58.4-DIN
- new net N$68: LED58.2-DOUT, LED59.4-DIN
- new net N$69: LED59.2-DOUT, LED60.4-DIN
- new net N$7: LED1.2-DOUT, LED2.4-DIN
- new net N$70: LED60.2-DOUT, LED61.4-DIN
- new net N$72: LED61.2-DOUT, LED62.4-DIN
- new net N$73: LED62.2-DOUT, LED63.4-DIN
- new net N$74: LED63.2-DOUT, LED64.4-DIN
- new net N$75: LED64.2-DOUT, LED65.4-DIN
- new net N$76: LED65.2-DOUT, LED66.4-DIN
- new net N$77: LED66.2-DOUT, LED67.4-DIN
- new net N$78: LED67.2-DOUT, LED68.4-DIN
- new net N$79: LED68.2-DOUT, LED69.4-DIN
- new net N$8: D4.A, R11.1
- new net N$80: LED69.2-DOUT, LED70.4-DIN
- new net N$81: LED70.2-DOUT, LED71.4-DIN
- new net N$82: LED71.2-DOUT, LED72.4-DIN
- new net N$83: LED72.2-DOUT, LED73.4-DIN
- new net N$85: LED73.2-DOUT, LED74.4-DIN
- new net N$86: LED74.2-DOUT, LED75.4-DIN
- new net N$87: LED75.2-DOUT, LED76.4-DIN
- new net N$88: LED76.2-DOUT, LED77.4-DIN
- new net N$89: LED77.2-DOUT, LED78.4-DIN
- new net N$90: LED78.2-DOUT, LED79.4-DIN
- new net N$91: LED79.2-DOUT, LED80.4-DIN
- new net N$92: LED80.2-DOUT, LED81.4-DIN
- new net N$93: LED81.2-DOUT, LED82.4-DIN
- new net N$94: LED82.2-DOUT, LED83.4-DIN
- new net N$95: LED83.2-DOUT, LED84.4-DIN
- new net N$96: LED84.2-DOUT, LED85.4-DIN
- new net N$98: LED85.2-DOUT, LED86.4-DIN
- new net N$99: LED86.2-DOUT, LED87.4-DIN
- new net PB1: S2.1, U1.31
- new net PB2: S3.1, U1.27
- new net PB3: S4.1, U1.1
- new net RXLED: R11.2, U1.8
- new net SCL: IC4.16, U1.18
- new net SDA: IC4.15, U1.19
- new net SEROUT: LED1.4-DIN, U1.25
- new net USBD+: JP2.D+, R6.1
- new net USBD-: JP2.D-, R7.1
- new net VBAT: G1.+, IC4.14
- new net VBUS: F1.2, JP2.VBUS
- new net VCAP: C11.+, U1.6
- net AREF: now also C10.1, U1.42; no longer C5.1, U$4.42
- net D+: now also R6.2, U1.4; no longer J1.D+, R3.2
- net D-: now also R7.2, U1.3; no longer J1.D-, R4.2
- net GATE_CMD: now also IC3.1, Q1.2; no longer IC6.1, Q1.G
- net GND: now also C11.-, C12.2, C13.-, C14.1, C15.1, C4.2, C5.-, C6.2, C8.2, D1.A, D3.C, D4.C, IC3.4, IC4.11, IC4.12, IC4.13, IC4.5, IC4.6, IC4.7, IC4.8, IC4.9, IC5.2, JP2.GND, JP3.6, JP4.2, LED1.3-GND, LED10.3-GND, LED100.3-GND, LED101.3-GND, LED102.3-GND, LED103.3-GND, LED104.3-GND, LED105.3-GND, LED106.3-GND, LED107.3-GND, LED108.3-GND, LED109.3-GND, LED11.3-GND, LED110.3-GND, LED111.3-GND, LED112.3-GND, LED113.3-GND, LED114.3-GND, LED115.3-GND, LED116.3-GND, LED117.3-GND, LED118.3-GND, LED119.3-GND, LED12.3-GND, LED120.3-GND, LED121.3-GND, LED122.3-GND, LED123.3-GND, LED124.3-GND, LED125.3-GND, LED126.3-GND, LED127.3-GND, LED128.3-GND, LED129.3-GND, LED13.3-GND, LED130.3-GND, LED131.3-GND, LED132.3-GND, LED133.3-GND, LED134.3-GND, LED135.3-GND, LED136.3-GND, LED137.3-GND, LED138.3-GND, LED139.3-GND, LED14.3-GND, LED140.3-GND, LED141.3-GND, LED142.3-GND, LED143.3-GND, LED144.3-GND, LED15.3-GND, LED16.3-GND, LED17.3-GND, LED18.3-GND, LED19.3-GND, LED2.3-GND, LED20.3-GND, LED21.3-GND, LED22.3-GND, LED23.3-GND, LED24.3-GND, LED25.3-GND, LED26.3-GND, LED27.3-GND, LED28.3-GND, LED29.3-GND, LED3.3-GND, LED30.3-GND, LED31.3-GND, LED32.3-GND, LED33.3-GND, LED34.3-GND, LED35.3-GND, LED36.3-GND, LED37.3-GND, LED38.3-GND, LED39.3-GND, LED4.3-GND, LED40.3-GND, LED41.3-GND, LED42.3-GND, LED43.3-GND, LED44.3-GND, LED45.3-GND, LED46.3-GND, LED47.3-GND, LED48.3-GND, LED49.3-GND, LED5.3-GND, LED50.3-GND, LED51.3-GND, LED52.3-GND, LED53.3-GND, LED54.3-GND, LED55.3-GND, LED56.3-GND, LED57.3-GND, LED58.3-GND, LED59.3-GND, LED6.3-GND, LED60.3-GND, LED61.3-GND, LED62.3-GND, LED63.3-GND, LED64.3-GND, LED65.3-GND, LED66.3-GND, LED67.3-GND, LED68.3-GND, LED69.3-GND, LED7.3-GND, LED70.3-GND, LED71.3-GND, LED72.3-GND, LED73.3-GND, LED74.3-GND, LED75.3-GND, LED76.3-GND, LED77.3-GND, LED78.3-GND, LED79.3-GND, LED8.3-GND, LED80.3-GND, LED81.3-GND, LED82.3-GND, LED83.3-GND, LED84.3-GND, LED85.3-GND, LED86.3-GND, LED87.3-GND, LED88.3-GND, LED89.3-GND, LED9.3-GND, LED90.3-GND, LED91.3-GND, LED92.3-GND, LED93.3-GND, LED94.3-GND, LED95.3-GND, LED96.3-GND, LED97.3-GND, LED98.3-GND, LED99.3-GND, R2.2, R9.2, S1.3, S2.2, S3.2, S4.2, U1.15, U1.23, U1.35, U1.43, U1.5; no longer C11.2, C12.1, C13.1, C14.-, C4.-, C5.2, C6.-, C8.1, D2.A, IC1.2, IC3.10, IC5.10, IC5.11, IC5.12, IC5.13, IC5.5, IC5.6, IC5.7, IC5.8, IC5.9, IC6.4, J1.GND, J4.6, JP1.PWR, R14.1, R6.1, R7.1, R8.1, S1.1, U$4.15, U$4.23, U$4.35, U$4.43, U$4.5, U1.22, U1.27, U2.22, U2.27, U3.22, U3.27
- net HWB: now also R9.1, U1.33; no longer R6.2, U$4.33
- net MISO: now also JP3.1; no longer J4.1, U$4.11
- net MOSI: now also JP3.4; no longer J4.4, U$4.10, U1.26
- net N$1: now also C6.1, IC3.3, R1.2, R2.1; no longer R5.2, U1.20
- net N$2: now also C14.2, R8.2, U1.17, Y1.2; no longer G1.+, IC5.14
- net N$3: now also C15.2, R8.1, U1.16, Y1.1; no longer R7.2, U2.20
- net N$4: now also R4.2, R5.2, U1.41; no longer R8.2, U3.20
- net RESET: now also D2.A, JP3.5, R3.1, S1.1, U1.13; no longer D1.A, J4.5, R1.2, S1.3, U$4.13
- net SCK: now also JP3.3; no longer J4.3, U$4.9, U1.25, U2.25, U3.25
- net TXLED: now also R10.2, U1.22; no longer U$4.22
- net VIN: now also D1.C, IC5.1, JP4.1, LED1.1-VDD, LED10.1-VDD, LED100.1-VDD, LED101.1-VDD, LED102.1-VDD, LED103.1-VDD, LED104.1-VDD, LED105.1-VDD, LED106.1-VDD, LED107.1-VDD, LED108.1-VDD, LED109.1-VDD, LED11.1-VDD, LED110.1-VDD, LED111.1-VDD, LED112.1-VDD, LED113.1-VDD, LED114.1-VDD, LED115.1-VDD, LED116.1-VDD, LED117.1-VDD, LED118.1-VDD, LED119.1-VDD, LED12.1-VDD, LED120.1-VDD, LED121.1-VDD, LED122.1-VDD, LED123.1-VDD, LED124.1-VDD, LED125.1-VDD, LED126.1-VDD, LED127.1-VDD, LED128.1-VDD, LED129.1-VDD, LED13.1-VDD, LED130.1-VDD, LED131.1-VDD, LED132.1-VDD, LED133.1-VDD, LED134.1-VDD, LED135.1-VDD, LED136.1-VDD, LED137.1-VDD, LED138.1-VDD, LED139.1-VDD, LED14.1-VDD, LED140.1-VDD, LED141.1-VDD, LED142.1-VDD, LED143.1-VDD, LED144.1-VDD, LED15.1-VDD, LED16.1-VDD, LED17.1-VDD, LED18.1-VDD, LED19.1-VDD, LED2.1-VDD, LED20.1-VDD, LED21.1-VDD, LED22.1-VDD, LED23.1-VDD, LED24.1-VDD, LED25.1-VDD, LED26.1-VDD, LED27.1-VDD, LED28.1-VDD, LED29.1-VDD, LED3.1-VDD, LED30.1-VDD, LED31.1-VDD, LED32.1-VDD, LED33.1-VDD, LED34.1-VDD, LED35.1-VDD, LED36.1-VDD, LED37.1-VDD, LED38.1-VDD, LED39.1-VDD, LED4.1-VDD, LED40.1-VDD, LED41.1-VDD, LED42.1-VDD, LED43.1-VDD, LED44.1-VDD, LED45.1-VDD, LED46.1-VDD, LED47.1-VDD, LED48.1-VDD, LED49.1-VDD, LED5.1-VDD, LED50.1-VDD, LED51.1-VDD, LED52.1-VDD, LED53.1-VDD, LED54.1-VDD, LED55.1-VDD, LED56.1-VDD, LED57.1-VDD, LED58.1-VDD, LED59.1-VDD, LED6.1-VDD, LED60.1-VDD, LED61.1-VDD, LED62.1-VDD, LED63.1-VDD, LED64.1-VDD, LED65.1-VDD, LED66.1-VDD, LED67.1-VDD, LED68.1-VDD, LED69.1-VDD, LED7.1-VDD, LED70.1-VDD, LED71.1-VDD, LED72.1-VDD, LED73.1-VDD, LED74.1-VDD, LED75.1-VDD, LED76.1-VDD, LED77.1-VDD, LED78.1-VDD, LED79.1-VDD, LED8.1-VDD, LED80.1-VDD, LED81.1-VDD, LED82.1-VDD, LED83.1-VDD, LED84.1-VDD, LED85.1-VDD, LED86.1-VDD, LED87.1-VDD, LED88.1-VDD, LED89.1-VDD, LED9.1-VDD, LED90.1-VDD, LED91.1-VDD, LED92.1-VDD, LED93.1-VDD, LED94.1-VDD, LED95.1-VDD, LED96.1-VDD, LED97.1-VDD, LED98.1-VDD, LED99.1-VDD, R1.1; no longer D2.C, IC1.1, IC3.9, IC4.9, JP1.GND, R10.1, R11.1, R12.1, R13.2, U1.19, U1.21, U2.19, U2.21, U3.19, U3.21
- net VUSB: now also C12.1, C13.+, F1.1, Q1.1, U1.7; no longer C14.+, C9.1, F1.2, Q1.D, U$4.7
Routing:
- net VIN: track 0.00 -> 2796.5 mm
- net R6: track 358.4 -> 0.00 mm, vias 12 -> 0
- net R12: track 358.1 -> 0.00 mm, vias 12 -> 0
- net R11: track 341.8 -> 0.00 mm, vias 12 -> 0
- net R5: track 341.2 -> 0.00 mm, vias 12 -> 0
- net R1: track 341.2 -> 0.00 mm, vias 12 -> 0
- net R7: track 338.8 -> 0.00 mm, vias 12 -> 0
- net R4: track 325.2 -> 0.00 mm, vias 12 -> 0
- net R2: track 324.6 -> 0.00 mm, vias 12 -> 0
- net R10: track 324.0 -> 0.00 mm, vias 12 -> 0
- net R8: track 321.1 -> 0.00 mm, vias 12 -> 0
- net R9: track 308.0 -> 0.00 mm, vias 12 -> 0
- net R3: track 308.0 -> 0.00 mm, vias 12 -> 0
- net C8RED: track 304.3 -> 0.00 mm
- net C4RED: track 304.3 -> 0.00 mm
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Other:
- board size 280 x 280 mm -> 230 x 230 mm
