File: Eagle/Word-Clock.brd (EAGLE design)
At the start: 230 x 230 mm, 196 parts, among them IC2 LM2936Z-3.3, IC3 LM358N, IC4 DS3231/SO, IC5 LM340H-05, Q1 PFETBS250, U1 ATMEGA32U4TQFP-44, Y1 16MHz

Commit message: Power Consumption Calculations
Parts:
- removed IC2: LM2936Z-3.3, national-semiconductor:TO92
- added C16: 100uF, resistor:C1210
- added C17, C18, C19, C20, C8: 100nF, resistor:C1206
- added D5: M7, diode:DO-214AC
- added D6: BLUETOOTH, led:CHIPLED_1206
- added IC1: LM340H-05, linear:TO220H
- added JP10, JP7, JP8, JP9: (no value), pinhead:1X03/90
- added JP11, JP12: (no value), SparkFun-Connectors:MOLEX-1X2
- added R18, R19, R20, R22: 1K, resistor:M1206
- added R21, R23, R24, R25, R26: 10K, resistor:M1206
- added R27, R28, R29, R30: 100K, resistor:M1206
- added R31, R32, R33, R34: 1M, resistor:M1206
- added S2: SWITCH-MOMENTARY-2SMD, SparkFun-Electromechanical:TACTILE-SWITCH-SMD
- added T1, T2: (no value), transistor:SOT23-BEC
- added U$1: LM3480IM4, SparkFun-PowerIC:SOT23-3
- added U$2: USB-PWR, adafruit:USB-MINIB-THM-MOLEX-PWRONLY
- added U2: ATMEGA32U4QFN2, SparkFun-DigitalIC:QFN-44-NOPAD
- added U3: HC_05, SerialPortBluetooth:BLUETOOTH_SMD
- added U4, U5, U6, U7: AT42QT1012, SparkFun-Sensors:SOT-23-6
- C1, C11, C13, C3, C5: device resistor:E2,5-6 -> resistor:C1210
- C10, C12, C2, C4, C6, C7, C9: device capacitor-wima:C5B2.5 -> resistor:C1206
- C14, C15: device resistor:C050-024X044 -> resistor:C1206
- D1: value 1N4001 -> M7; device diode:DO41-10 -> diode:DO-214AC
- D2: device diode:DO35-7 -> diode:SOD-123_MINI-SMA
- D3: value (none) -> RED; device SparkFun-LED:LED-1206 -> led:CHIPLED_1206
- D4: value (none) -> BLUE; device SparkFun-LED:LED-1206 -> led:CHIPLED_1206
- I1: device rcl:0207/7 -> rcl:L3216C
- IC3: value LM358N -> LM358D; device linear:DIL08 -> linear:SO08
- JP1: device SparkFun-Connectors:2X3-SHROUDED -> pinhead:1X06/90
- JP2: value USBPTH-VERTICAL -> USB-MICROB; device SparkFun-Connectors:USB-B-PTH-VERTICAL -> adafruit:USB-MINIB-THM-MOLEX
- JP3: device SparkFun-Connectors:2X3-SHROUDED -> pinhead:2X03/90
- Q1: value PFETBS250 -> FDN360P; device adafruit:TO92-OVAL -> transistor-power:SUPER-SOT3
- R1, R10, R11, R13, R15, R17, R2, R3, R5, R6, R7, R8, R9: device resistor:0207/7 -> resistor:M1206
- S1: value (none) -> SWITCH-MOMENTARY-2SMD; device SparkFun-Electromechanical:TACTILE-PTH -> SparkFun-Electromechanical:TACTILE-SWITCH-SMD
- Y1: device SparkFun-FreqCtrl:HC49U-V -> SparkFun-FreqCtrl:HC49UP
- moved R15 341.0 mm to (201.0, 194.0), flipped to the bottom
- moved R14 340.2 mm to (201.0, 199.0)
- moved R13 269.3 mm to (40.0, 194.0), flipped to the bottom
- moved R12 267.5 mm to (40.0, 199.0)
- moved R16 235.6 mm to (200.0, 40.0)
- moved R17 235.5 mm to (200.0, 35.0), flipped to the bottom
- moved JP5 178.1 mm to (3.00, 66.0), flipped to the bottom, turned to 90 degrees
- moved JP6 171.5 mm to (3.00, 59.0), flipped to the bottom, turned to 90 degrees
- moved JP2 114.4 mm to (240.0, 120.0), turned to 270 degrees
- moved R4 110.0 mm to (40.0, 39.0), flipped to the top, turned to 0 degrees
- moved G1 108.7 mm to (109.0, 32.0), turned to 90 degrees
- moved R2 102.4 mm to (161.0, 82.0), turned to 180 degrees
- moved C6 102.1 mm to (161.0, 79.0), turned to 180 degrees
- moved R1 97.1 mm to (161.0, 76.0), turned to 0 degrees
- moved C5 81.3 mm to (117.0, 81.0)
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Connections:
- removed net N$2 (its old number): C14.2, R8.2, U1.17, Y1.2
- removed net SW_L: JP5.1, U1.31
- removed net SW_R: JP6.1, U1.27
- new net A4: U1.40, U2.40
- new net A5: U1.41, U2.41
- new net D11: U1.12, U2.12
- new net D12: U1.26, U2.26
- new net D13: U1.32, U2.32
- new net D5: U1.31, U2.31
- new net D7: U1.1, U2.1
- new net N$110: C19.1, R23.2, U5.3
- new net N$136: C18.1, R24.2, U4.3
- new net N$149: C17.1, R25.2, U6.3
- new net N$161: C19.2, R34.1, U5.4
- new net N$162: C18.2, R31.1, U4.4
- new net N$163: C17.2, R32.1, U6.4
- new net N$164: JP7.2, U4.6
- new net N$165: JP8.2, U5.6
- new net N$166: JP10.2, U7.6
- new net N$167: JP9.2, U6.6
- new net N$32: R22.1, U3.33
- new net N$4: R19.1, T1.C, T2.B
- new net N$45: D6.A, R22.2
- new net N$84: C20.1, R26.2, U7.3
- new net N$9: R21.1, S2.1, U3.34
- new net N$97: C20.2, R33.1, U7.4
- new net PAD1: R24.1
- new net PAD2: R23.1
- new net PAD3: R25.1
- new net PAD4: R26.1
- new net SW_1: JP5.1, R28.2, U1.27, U2.27, U4.1
- new net SW_2: JP6.1, R27.2, U1.28, U2.28, U5.1
- new net SW_3: JP11.1, R29.2, U1.29, U2.29, U6.1
- new net SW_4: JP12.1, R30.2, U1.30, U2.30, U7.1
- new net UART_RXD: D5.A, U3.2
- new net UART_TXD: R18.2, U3.1
- new net VCC: C16.1, C7.1, C8.1, D2.C, I1.1, IC1.3, Q1.2, R3.2, U1.14, U1.2, U1.24, U1.34, U2.14, U2.2, U2.24, U2.34
- new net XTAL1: C14.2, R8.2, U1.17, U2.17, Y1.2
- new net XTAL2: C15.2, R8.1, U1.16, U2.16, Y1.1
- net 3.3V: now also C4.2, C5.1, R19.2, S2.3, U$1.1, U3.12; no longer C4.1, C5.+, IC2.1
- net 5V: now also C3.1, JP10.1, JP7.1, JP8.1, JP9.1, LED1.1-VDD, LED10.1-VDD, LED100.1-VDD, LED101.1-VDD, LED102.1-VDD, LED103.1-VDD, LED104.1-VDD, LED105.1-VDD, LED106.1-VDD, LED107.1-VDD, LED108.1-VDD, LED109.1-VDD, LED11.1-VDD, LED110.1-VDD, LED111.1-VDD, LED112.1-VDD, LED113.1-VDD, LED114.1-VDD, LED115.1-VDD, LED116.1-VDD, LED117.1-VDD, LED118.1-VDD, LED119.1-VDD, LED12.1-VDD, LED120.1-VDD, LED121.1-VDD, LED122.1-VDD, LED123.1-VDD, LED124.1-VDD, LED125.1-VDD, LED126.1-VDD, LED127.1-VDD, LED128.1-VDD, LED129.1-VDD, LED13.1-VDD, LED130.1-VDD, LED131.1-VDD, LED132.1-VDD, LED133.1-VDD, LED134.1-VDD, LED135.1-VDD, LED136.1-VDD, LED137.1-VDD, LED138.1-VDD, LED139.1-VDD, LED14.1-VDD, LED140.1-VDD, LED141.1-VDD, LED142.1-VDD, LED143.1-VDD, LED144.1-VDD, LED15.1-VDD, LED16.1-VDD, LED17.1-VDD, LED18.1-VDD, LED19.1-VDD, LED2.1-VDD, LED20.1-VDD, LED21.1-VDD, LED22.1-VDD, LED23.1-VDD, LED24.1-VDD, LED25.1-VDD, LED26.1-VDD, LED27.1-VDD, LED28.1-VDD, LED29.1-VDD, LED3.1-VDD, LED30.1-VDD, LED31.1-VDD, LED32.1-VDD, LED33.1-VDD, LED34.1-VDD, LED35.1-VDD, LED36.1-VDD, LED37.1-VDD, LED38.1-VDD, LED39.1-VDD, LED4.1-VDD, LED40.1-VDD, LED41.1-VDD, LED42.1-VDD, LED43.1-VDD, LED44.1-VDD, LED45.1-VDD, LED46.1-VDD, LED47.1-VDD, LED48.1-VDD, LED49.1-VDD, LED5.1-VDD, LED50.1-VDD, LED51.1-VDD, LED52.1-VDD, LED53.1-VDD, LED54.1-VDD, LED55.1-VDD, LED56.1-VDD, LED57.1-VDD, LED58.1-VDD, LED59.1-VDD, LED6.1-VDD, LED60.1-VDD, LED61.1-VDD, LED62.1-VDD, LED63.1-VDD, LED64.1-VDD, LED65.1-VDD, LED66.1-VDD, LED67.1-VDD, LED68.1-VDD, LED69.1-VDD, LED7.1-VDD, LED70.1-VDD, LED71.1-VDD, LED72.1-VDD, LED73.1-VDD, LED74.1-VDD, LED75.1-VDD, LED76.1-VDD, LED77.1-VDD, LED78.1-VDD, LED79.1-VDD, LED8.1-VDD, LED80.1-VDD, LED81.1-VDD, LED82.1-VDD, LED83.1-VDD, LED84.1-VDD, LED85.1-VDD, LED86.1-VDD, LED87.1-VDD, LED88.1-VDD, LED89.1-VDD, LED9.1-VDD, LED90.1-VDD, LED91.1-VDD, LED92.1-VDD, LED93.1-VDD, LED94.1-VDD, LED95.1-VDD, LED96.1-VDD, LED97.1-VDD, LED98.1-VDD, LED99.1-VDD, R20.1, R27.1, R28.1, R29.1, R30.1, R31.2, R32.2, R33.2, R34.2, U$1.2, U4.5, U5.5, U6.5, U7.5; no longer C3.+, C7.1, D2.C, I1.1, IC2.3, Q1.3, R3.2, U1.14, U1.2, U1.24, U1.34
- net AREF: now also U2.42
- net AVCC: now also U2.44
- net D+: now also U2.4
- net D-: now also U2.3
- net GATE_CMD: now also Q1.1; no longer Q1.2
- net GND: now also C1.2, C11.2, C13.2, C16.2, C3.2, C4.1, C5.2, C8.2, D6.C, IC1.2, JP10.3, JP11.2, JP12.2, JP7.3, JP8.3, JP9.3, R21.2, T1.E, T2.E, U$1.3, U$2.GND, U2.15, U2.23, U2.35, U2.43, U2.5, U3.13, U3.21, U3.22, U4.2, U5.2, U6.2, U7.2; no longer C1.-, C11.-, C13.-, C3.-, C4.2, C5.-, IC2.2
- net HWB: now also U2.33
- net LDR1_PIN: now also U2.36
- net LDR2_PIN: now also U2.37
- net LDR3_PIN: now also U2.38
- net LDR4_PIN: now also U2.39
- net MISO: now also U2.11
- net MOSI: now also U2.10
- net N$3: now also R18.1, T1.B; no longer C15.2, R8.1, U1.16, Y1.1
- net N$6: now also R10.2; no longer R10.1
- net RESET: now also U2.13
- net RXD: now also R20.2, T2.C, U2.20
- net RXLED: now also U2.8
- net SCK: now also U2.9
- net SCL: now also U2.18
- net SDA: now also U2.19
- net SEROUT: now also U2.25
- net TXD: now also D5.C, U2.21
- net TXLED: now also R10.1, U2.22; no longer R10.2
- net VCAP: now also C11.1, U2.6; no longer C11.+
- net VIN: now also C1.1, IC1.1, U$2.VBUS; no longer C1.+, LED1.1-VDD, LED10.1-VDD, LED100.1-VDD, LED101.1-VDD, LED102.1-VDD, LED103.1-VDD, LED104.1-VDD, LED105.1-VDD, LED106.1-VDD, LED107.1-VDD, LED108.1-VDD, LED109.1-VDD, LED11.1-VDD, LED110.1-VDD, LED111.1-VDD, LED112.1-VDD, LED113.1-VDD, LED114.1-VDD, LED115.1-VDD, LED116.1-VDD, LED117.1-VDD, LED118.1-VDD, LED119.1-VDD, LED12.1-VDD, LED120.1-VDD, LED121.1-VDD, LED122.1-VDD, LED123.1-VDD, LED124.1-VDD, LED125.1-VDD, LED126.1-VDD, LED127.1-VDD, LED128.1-VDD, LED129.1-VDD, LED13.1-VDD, LED130.1-VDD, LED131.1-VDD, LED132.1-VDD, LED133.1-VDD, LED134.1-VDD, LED135.1-VDD, LED136.1-VDD, LED137.1-VDD, LED138.1-VDD, LED139.1-VDD, LED14.1-VDD, LED140.1-VDD, LED141.1-VDD, LED142.1-VDD, LED143.1-VDD, LED144.1-VDD, LED15.1-VDD, LED16.1-VDD, LED17.1-VDD, LED18.1-VDD, LED19.1-VDD, LED2.1-VDD, LED20.1-VDD, LED21.1-VDD, LED22.1-VDD, LED23.1-VDD, LED24.1-VDD, LED25.1-VDD, LED26.1-VDD, LED27.1-VDD, LED28.1-VDD, LED29.1-VDD, LED3.1-VDD, LED30.1-VDD, LED31.1-VDD, LED32.1-VDD, LED33.1-VDD, LED34.1-VDD, LED35.1-VDD, LED36.1-VDD, LED37.1-VDD, LED38.1-VDD, LED39.1-VDD, LED4.1-VDD, LED40.1-VDD, LED41.1-VDD, LED42.1-VDD, LED43.1-VDD, LED44.1-VDD, LED45.1-VDD, LED46.1-VDD, LED47.1-VDD, LED48.1-VDD, LED49.1-VDD, LED5.1-VDD, LED50.1-VDD, LED51.1-VDD, LED52.1-VDD, LED53.1-VDD, LED54.1-VDD, LED55.1-VDD, LED56.1-VDD, LED57.1-VDD, LED58.1-VDD, LED59.1-VDD, LED6.1-VDD, LED60.1-VDD, LED61.1-VDD, LED62.1-VDD, LED63.1-VDD, LED64.1-VDD, LED65.1-VDD, LED66.1-VDD, LED67.1-VDD, LED68.1-VDD, LED69.1-VDD, LED7.1-VDD, LED70.1-VDD, LED71.1-VDD, LED72.1-VDD, LED73.1-VDD, LED74.1-VDD, LED75.1-VDD, LED76.1-VDD, LED77.1-VDD, LED78.1-VDD, LED79.1-VDD, LED8.1-VDD, LED80.1-VDD, LED81.1-VDD, LED82.1-VDD, LED83.1-VDD, LED84.1-VDD, LED85.1-VDD, LED86.1-VDD, LED87.1-VDD, LED88.1-VDD, LED89.1-VDD, LED9.1-VDD, LED90.1-VDD, LED91.1-VDD, LED92.1-VDD, LED93.1-VDD, LED94.1-VDD, LED95.1-VDD, LED96.1-VDD, LED97.1-VDD, LED98.1-VDD, LED99.1-VDD
- net VUSB: now also C13.1, Q1.3, U2.7; no longer C13.+, Q1.1
Routing:
- net VIN: track 2812.0 -> 0.00 mm
- net 5V: track 263.4 -> 0.00 mm
- net N$96: track 199.3 -> 0.00 mm
- net N$83: track 199.3 -> 0.00 mm
- net N$70: track 199.3 -> 0.00 mm
- net N$57: track 199.3 -> 0.00 mm
- net N$44: track 199.3 -> 0.00 mm
- net N$31: track 199.3 -> 0.00 mm
- net N$19: track 199.3 -> 0.00 mm
- net N$148: track 199.3 -> 0.00 mm
- net N$135: track 199.3 -> 0.00 mm
- net N$122: track 199.3 -> 0.00 mm
- net N$109: track 199.3 -> 0.00 mm
- net USBD+: track 105.8 -> 0.00 mm
- net USBD-: track 101.4 -> 0.00 mm
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Other:
- board size 230 x 230 mm -> 240 x 240 mm

Commit message: V1.2 PCB
Parts:
- removed D2: 1N4148, diode:SOD-123_MINI-SMA
- removed D3: RED, led:CHIPLED_1206
- removed D4: BLUE, led:CHIPLED_1206
- removed F1: 500mA, adafruit:R1206
- removed G1: CR2032H, battery:CR2032H
- removed JP10, JP7, JP8, JP9: (no value), pinhead:1X03/90
- removed JP11, JP12, JP4, JP5, JP6: (no value), SparkFun-Connectors:MOLEX-1X2
- removed JP3: (no value), pinhead:2X03/90
- removed Q1: FDN360P, transistor-power:SUPER-SOT3
- removed R30: 100K, resistor:M1206
- removed R31, R32, R33, R34: 1M, resistor:M1206
- removed T2: (no value), transistor:SOT23-BEC
- removed U2: ATMEGA32U4QFN2, SparkFun-DigitalIC:QFN-44-NOPAD
- removed U5, U6, U7: AT42QT1012, SparkFun-Sensors:SOT-23-6
- added BLUETOOTH, DS3231: (no value), SparkFun-Connectors:1X06-SMD-FEMALE-V2
- added C21: 1u, resistor:SMC_A
- added C22, C23, C24, C25, C26, C27, C28, C29, C30, C31, C34: 100n, resistor:C1206
- added C32, C33: 10u, resistor:SMC_C
- added CN1, CN2: (no value), adafruit:USB-MINIB-THM
- added H1, H2, H3, H4: MOUNT-HOLE5.5, holes:5,5
- added IC2: LMV358IDGKR, linear:SO08
- added IC6: LP2985-33DBVR, SmartPrj:SOT23-DBV
- added J1, J2, J3, J4: 22-05-7028-02, con-molex:7395-02
- added L1: MH2029-300Y, wuerth-elektronik:0805
- added ONLED: BLUE, SparkFun-LED:LED-1206
- added PAD1A, PAD2A, PAD3A, PAD4A: (no value), wirepad:2,54/1,0
- added PAD1B, PAD2B, PAD3B, PAD4B: CAPSENSE_PAD, SparkFun-Electromechanical:CAPSENSE_PAD
- added RXLED: GREEN, SparkFun-LED:LED-1206
- added S10, S11, S12, S9: SWITCH-MOMENTARY-2TACTILE-SWITCH-SMD-RIGHT-ANGLE, SparkFun-Electromechanical:TACTILE_SWITCH-SMD-RIGHT-ANGLE
- added S3: SWITCH-MOMENTARY-2SMD-1101NE, SparkFun-Electromechanical:TACTILE-SWITCH-1101NE
- added S5, S6, S7, S8: (no value), SparkFun-Electromechanical:AYZ0202
- added TXLED: RED, SparkFun-LED:LED-1206
- added U$3, U$4, U$5: AT42QT1010SOT23, SparkFun-DigitalIC:SOT23-6
- added X1: (no value), adafruit:ESP-12
- added Z1, Z2: CG0603MLC-05E, varistor:CT/CN0603
- C1: value 100uF -> 100n; device resistor:C1210 -> resistor:C1206
- C10, C8, C9: value 100nF -> 10u; device resistor:C1206 -> resistor:SMC_C
- C11: value 1uF -> 100n; device resistor:C1210 -> resistor:C1206
- C12, C18, C19, C2, C6: value 100nF -> 100n
- C13: value 1uF -> 1u; device resistor:C1210 -> resistor:SMC_C
- C14: value 22pF -> 100n
- C15: value 22pF -> 1u; device resistor:C1206 -> resistor:SMC_C
- C16: value 100uF -> 1u; device resistor:C1210 -> resistor:SMC_A
- C17, C20: value 100nF -> 1u; device resistor:C1206 -> resistor:SMC_A
- C3: value 100uF -> 1uF; device resistor:C1210 -> resistor:SMC_C
- C4: value 100nF -> 1uF; device resistor:C1206 -> resistor:SMC_C
- C5: value 100uF -> 22p; device resistor:C1210 -> resistor:C1206
- C7: value 100nF -> 22p
- D1: value M7 -> CD1206-S01575; device diode:DO-214AC -> diode:MINIMELF
- D5: device diode:DO-214AC -> diode:SMB
- D6: value BLUETOOTH -> BLUE; device led:CHIPLED_1206 -> SparkFun-LED:LED-1206
- I1: value (none) -> MF-MSMF050-2 500mA; device rcl:L3216C -> rcl:L1812
- IC1: value LM340H-05 -> NCP1117ST50T3G; device linear:TO220H -> linear:SOT223
- IC3: value LM358D -> LP2985-33DBVR; device linear:SO08 -> SmartPrj:SOT23-DBV
- IC4: value DS3231/SO -> LP2985-33DBVR; device adafruit:SO16W -> SmartPrj:SOT23-DBV
- IC5: value LM340H-05 -> DS3231/SO; device linear:TO220H -> adafruit:SO16W
- JP1: device pinhead:1X06/90 -> pinhead:2X03/90
- JP2: value USB-MICROB -> POWER_JACKCOMBO; device adafruit:USB-MINIB-THM-MOLEX -> SparkFun-Connectors:POWER_JACK_COMBO
- R1, R3: value 10k -> 10K; device resistor:M1206 -> resistor:R1206
- R10: value 1K -> 22R; device resistor:M1206 -> resistor:R1206
- R11: value 1K -> 10K; device resistor:M1206 -> resistor:R1206
- R12: value PHOTOCELLPTH -> 10K; device SparkFun-Sensors:PHOTOCELL -> resistor:R1206
- R13: value 10k -> 470; device resistor:M1206 -> resistor:R1206
- R14, R16: value PHOTOCELLPTH -> 12K; device SparkFun-Sensors:PHOTOCELL -> resistor:R1206
- R15, R17: value 10k -> 22K; device resistor:M1206 -> resistor:R1206
- R18: value 1K -> 22K; device resistor:M1206 -> resistor:R1206
- R19, R20, R22: value 1K -> 12K; device resistor:M1206 -> resistor:R1206
- R2: value 10k -> 1M; device resistor:M1206 -> resistor:R1206
- R21, R25, R26: value 10K -> 12K; device resistor:M1206 -> resistor:R1206
- R23, R24: value 10K -> PHOTOCELLPTH; device resistor:M1206 -> SparkFun-Sensors:PHOTOCELL
- R27, R28: value 100K -> 12K; device resistor:M1206 -> resistor:R1206
- R29: value 100K -> 470; device resistor:M1206 -> resistor:R1206
- R5: value 10k -> PHOTOCELLPTH; device resistor:M1206 -> SparkFun-Sensors:PHOTOCELL
- R6, R7: value 22R -> 1K; device resistor:M1206 -> resistor:R1206
- R8: value 1M -> K; device resistor:M1206 -> resistor:R1206
- R9: value 10k -> 22R; device resistor:M1206 -> resistor:R1206
- S1, S2: value SWITCH-MOMENTARY-2SMD -> SWITCH-MOMENTARY-2SMD-1101NE; device SparkFun-Electromechanical:TACTILE-SWITCH-SMD -> SparkFun-Electromechanical:TACTILE-SWITCH-1101NE
- T1: value (none) -> FDN340P; device transistor:SOT23-BEC -> zetex:SOT-23
- U$1: value LM3480IM4 -> (none); device SparkFun-PowerIC:SOT23-3 -> adafruit:CR2032-SMD
- U$2: value USB-PWR -> AT42QT1010SOT23; device adafruit:USB-MINIB-THM-MOLEX-PWRONLY -> SparkFun-DigitalIC:SOT23-6
- U4: value AT42QT1012 -> +12v; device SparkFun-Sensors:SOT-23-6 -> SparkFun-PowerIC:TO-252
- moved R24 318.8 mm to (20.0, 240.0)
- moved R21 313.2 mm to (295.0, 12.0), flipped to the top
- moved R4 313.1 mm to (280.0, 240.0), flipped to the bottom
- moved R28 312.7 mm to (164.0, 101.0), flipped to the top, turned to 270 degrees
- moved C19 311.7 mm to (197.2, 83.9), flipped to the top, turned to 180 degrees
- moved R27 304.9 mm to (160.0, 101.0), flipped to the top, turned to 270 degrees
- moved C18 303.0 mm to (197.2, 76.3), flipped to the top
- moved C17 301.9 mm to (197.2, 81.4), flipped to the top, turned to 180 degrees
- moved R29 300.9 mm to (144.0, 96.0), flipped to the top, turned to 90 degrees
- moved R26 289.6 mm to (172.0, 101.0), flipped to the top, turned to 270 degrees
- moved R25 282.1 mm to (168.0, 101.0), flipped to the top, turned to 270 degrees
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Connections:
- removed net 3.3V: C4.2, C5.1, IC3.2, R19.2, S2.3, U$1.1, U3.12
- removed net 5V: C2.1, C3.1, IC3.8, IC4.2, IC5.3, JP1.3, JP10.1, JP3.2, JP7.1, JP8.1, JP9.1, LED1.1-VDD, LED10.1-VDD, LED100.1-VDD, LED101.1-VDD, LED102.1-VDD, LED103.1-VDD, LED104.1-VDD, LED105.1-VDD, LED106.1-VDD, LED107.1-VDD, LED108.1-VDD, LED109.1-VDD, LED11.1-VDD, LED110.1-VDD, LED111.1-VDD, LED112.1-VDD, LED113.1-VDD, LED114.1-VDD, LED115.1-VDD, LED116.1-VDD, LED117.1-VDD, LED118.1-VDD, LED119.1-VDD, LED12.1-VDD, LED120.1-VDD, LED121.1-VDD, LED122.1-VDD, LED123.1-VDD, LED124.1-VDD, LED125.1-VDD, LED126.1-VDD, LED127.1-VDD, LED128.1-VDD, LED129.1-VDD, LED13.1-VDD, LED130.1-VDD, LED131.1-VDD, LED132.1-VDD, LED133.1-VDD, LED134.1-VDD, LED135.1-VDD, LED136.1-VDD, LED137.1-VDD, LED138.1-VDD, LED139.1-VDD, LED14.1-VDD, LED140.1-VDD, LED141.1-VDD, LED142.1-VDD, LED143.1-VDD, LED144.1-VDD, LED15.1-VDD, LED16.1-VDD, LED17.1-VDD, LED18.1-VDD, LED19.1-VDD, LED2.1-VDD, LED20.1-VDD, LED21.1-VDD, LED22.1-VDD, LED23.1-VDD, LED24.1-VDD, LED25.1-VDD, LED26.1-VDD, LED27.1-VDD, LED28.1-VDD, LED29.1-VDD, LED3.1-VDD, LED30.1-VDD, LED31.1-VDD, LED32.1-VDD, LED33.1-VDD, LED34.1-VDD, LED35.1-VDD, LED36.1-VDD, LED37.1-VDD, LED38.1-VDD, LED39.1-VDD, LED4.1-VDD, LED40.1-VDD, LED41.1-VDD, LED42.1-VDD, LED43.1-VDD, LED44.1-VDD, LED45.1-VDD, LED46.1-VDD, LED47.1-VDD, LED48.1-VDD, LED49.1-VDD, LED5.1-VDD, LED50.1-VDD, LED51.1-VDD, LED52.1-VDD, LED53.1-VDD, LED54.1-VDD, LED55.1-VDD, LED56.1-VDD, LED57.1-VDD, LED58.1-VDD, LED59.1-VDD, LED6.1-VDD, LED60.1-VDD, LED61.1-VDD, LED62.1-VDD, LED63.1-VDD, LED64.1-VDD, LED65.1-VDD, LED66.1-VDD, LED67.1-VDD, LED68.1-VDD, LED69.1-VDD, LED7.1-VDD, LED70.1-VDD, LED71.1-VDD, LED72.1-VDD, LED73.1-VDD, LED74.1-VDD, LED75.1-VDD, LED76.1-VDD, LED77.1-VDD, LED78.1-VDD, LED79.1-VDD, LED8.1-VDD, LED80.1-VDD, LED81.1-VDD, LED82.1-VDD, LED83.1-VDD, LED84.1-VDD, LED85.1-VDD, LED86.1-VDD, LED87.1-VDD, LED88.1-VDD, LED89.1-VDD, LED9.1-VDD, LED90.1-VDD, LED91.1-VDD, LED92.1-VDD, LED93.1-VDD, LED94.1-VDD, LED95.1-VDD, LED96.1-VDD, LED97.1-VDD, LED98.1-VDD, LED99.1-VDD, R12.1, R14.1, R16.1, R20.1, R27.1, R28.1, R29.1, R30.1, R31.2, R32.2, R33.2, R34.2, R4.1, U$1.2, U4.5, U5.5, U6.5, U7.5
- removed net D11: U1.12, U2.12
- removed net D12: U1.26, U2.26
- removed net D13: U1.32, U2.32
- removed net D5: U1.31, U2.31
- removed net LDR1_PIN: R4.2, R5.2, U1.36, U2.36
- removed net LDR2_PIN: R12.2, R13.2, U1.37, U2.37
- removed net LDR3_PIN: R14.2, R15.2, U1.38, U2.38
- removed net LDR4_PIN: R16.2, R17.2, U1.39, U2.39
- removed net N$110 (its old number): C19.1, R23.2, U5.3
- removed net N$136 (its old number): C18.1, R24.2, U4.3
- removed net N$149: C17.1, R25.2, U6.3
- removed net N$161: C19.2, R34.1, U5.4
- removed net N$162: C18.2, R31.1, U4.4
- removed net N$163: C17.2, R32.1, U6.4
- removed net N$164: JP7.2, U4.6
- removed net N$165: JP8.2, U5.6
- removed net N$166: JP10.2, U7.6
- removed net N$167: JP9.2, U6.6
- removed net N$32 (its old number): R22.1, U3.33
- removed net N$4 (its old number): R19.1, T1.C, T2.B
- removed net N$45 (its old number): D6.A, R22.2
- removed net N$6 (its old number): D3.A, R10.2
- removed net N$8 (its old number): D4.A, R11.1
- removed net N$84 (its old number): C20.1, R26.2, U7.3
- removed net N$9 (its old number): R21.1, S2.1, U3.34
- removed net N$97 (its old number): C20.2, R33.1, U7.4
- removed net RXD: JP1.4, R20.2, T2.C, U1.20, U2.20
- removed net SCL: IC4.16, U1.18, U2.18
- removed net SDA: IC4.15, U1.19, U2.19
- removed net SEROUT: LED1.4-DIN, U1.25, U2.25
- removed net SW_1: JP5.1, R28.2, U1.27, U2.27, U4.1
- removed net SW_2: JP6.1, R27.2, U1.28, U2.28, U5.1
- removed net SW_3: JP11.1, R29.2, U1.29, U2.29, U6.1
- removed net SW_4: JP12.1, R30.2, U1.30, U2.30, U7.1
- removed net TXD: D5.C, JP1.5, U1.21, U2.21
- removed net UART_RXD: D5.A, U3.2
- removed net UART_TXD: R18.2, U3.1
- removed net USBD+: JP2.D+, R6.1
- removed net USBD-: JP2.D-, R7.1
- removed net VBUS: F1.2, JP2.VBUS
- removed net VCAP: C11.1, U1.6, U2.6
- new net +3V3: C13.-, IC2.6, IC3.5
- new net +3V3B: C17.-, C19.2, IC4.5, U3.12
- new net +3V3C: C21.-, C23.2, IC6.5, R18.2, X1.8
- new net +5V: BLUETOOTH.5, C1.1, C12.1, C15.-, C16.-, C18.2, C2.1, C20.-, C22.2, C8.+, D1.C, DS3231.5, IC1.2, IC1.4, IC2.8, IC3.1, IC3.3, IC4.1, IC4.3, IC5.2, IC6.1, IC6.3, JP1.2, L1.1, R1.2, R23.2, R24.2, R4.2, R5.2, R6.2, R7.2, R8.2, S5.1, S6.1, S7.1, S8.1, T1.2, U$2.5, U$3.5, U$4.5, U$5.5, U1.14, U1.2, U1.34
- new net A0: J3.1, S10.1, U1.36
- new net A1: J4.1, S9.1, U1.37
- new net A2: R26.2, R5.1, U1.38
- new net A3: R25.2, R4.1, U1.39
- new net BLUETOOTHLED: D6.A, R13.2
- new net CMP: C14.2, IC2.5, R11.1, R12.2
- new net D0/RX: U1.20, X1.16
- new net D1/TX: R16.1, R17.1, U1.21
- new net D2/SDA: DS3231.4, IC5.15, U1.19
- new net D3/SCL: DS3231.3, IC5.16, U1.18
- new net D4: U$5.1, U1.25
- new net D5*: J1.1, S12.1, U1.31
- new net D6*: U$3.1, U1.27
- new net DS3231RST: IC5.4, S3.2
- new net ESP12RESET: R18.1, S2.2, X1.1
- new net ESP12RX: R16.2, X1.15
- new net HC-05RX: R14.2, U3.2
- new net IO10*: BLUETOOTH.3, U1.30, U3.1
- new net IO11*: BLUETOOTH.2, R14.1, R15.2, U1.12
- new net IO12: U$2.1, U1.26
- new net IO13*: J2.1, S11.1, U1.32
- new net IO8: U$4.1, U1.28
- new net IO9*: BLUETOOTH.6, U1.29, U3.34
- new net MODE1: S7.2, U$4.6
- new net MODE2: S8.2, U$5.6
- new net MODE3: S5.2, U$2.6
- new net MODE4: S6.2, U$3.6
- new net N$147: LED1.4-DIN, R29.2
- new net N$2: R7.1, RXLED.A
- new net RD+: R9.2, U1.4
- new net RD-: R10.2, U1.3
- new net SNS1: C28.1, U$4.4
- new net SNS2: C30.1, U$5.4
- new net SNS3: C24.1, U$2.4
- new net SNS4: C26.1, U$3.4
- new net SNSK1: C28.2, R21.1, U$4.3
- new net SNSK2: C30.2, R22.1, U$5.3
- new net SNSK3: C24.2, R19.1, U$2.3
- new net SNSK4: C26.2, R20.1, U$3.3
- new net STATE: R13.1, U3.31
- new net UCAP: C4.+, U1.6
- new net USBID: CN1.ID
- new net XUSB: CN1.VBUS, I1.2
- net A4: now also R24.1, R28.2; no longer U2.40
- net A5: now also R23.1, R27.2; no longer U2.41
- net AREF: now also C6.2; no longer C10.1, U2.42
- net AVCC: now also C3.+, L1.2, U1.24; no longer C9.1, I1.2, U2.44
- net D+: now also CN1.D+, R9.1, Z1.1; no longer R6.2, U1.4, U2.4
- net D-: now also CN1.D-, R10.1, Z2.1; no longer R7.2, U1.3, U2.3
- net D7: now also R29.1; no longer U2.1
- net GATE_CMD: now also IC2.7, T1.3; no longer IC3.1, Q1.1
- net GND: now also BLUETOOTH.4, C10.-, C11.1, C13.+, C15.+, C16.+, C17.+, C18.1, C19.1, C20.+, C21.+, C22.1, C23.1, C25.1, C27.1, C29.1, C3.-, C31.1, C32.-, C33.-, C34.2, C4.-, C5.1, C6.1, C8.-, C9.-, CN1.GND, CN2.GND, D5.A, DS3231.6, IC1.1, IC2.4, IC3.2, IC4.2, IC5.10, IC5.11, IC5.12, IC5.13, IC5.5, IC5.6, IC5.7, IC5.8, IC5.9, IC6.2, J1.2, J2.2, J3.2, J4.2, JP1.6, JP2.GND@1, ONLED.C, R12.1, R17.2, R25.1, R26.1, R27.1, R28.1, R3.2, S1.2, S10.2, S11.2, S12.2, S2.1, S3.1, S5.3, S6.3, S7.3, S8.3, S9.2, U$1.-, U$2.2, U$3.2, U$4.2, U$5.2, U4.3, X1.9, Z1.2, Z2.2; no longer C10.2, C11.2, C13.2, C15.1, C16.2, C3.2, C4.1, C5.2, C6.2, C8.2, C9.2, D1.A, D3.C, D4.C, G1.-, IC1.2, IC3.4, IC4.10, IC4.11, IC4.12, IC4.13, IC4.5, IC4.6, IC4.7, IC4.8, IC4.9, IC5.2, JP1.1, JP1.2, JP10.3, JP11.2, JP12.2, JP3.6, JP4.2, JP5.2, JP6.2, JP7.3, JP8.3, JP9.3, R13.1, R17.1, R2.2, R21.2, R5.1, R9.2, S1.3, T1.E, T2.E, U$1.3, U$2.GND, U2.15, U2.23, U2.35, U2.43, U2.5, U4.2, U5.2, U6.2, U7.2
- net HWB: now also R3.1; no longer R9.1, U2.33
- net MISO: now also JP1.1; no longer JP3.1, U2.11
- net MOSI: now also JP1.4; no longer JP3.4, U2.10
- net N$1: now also R6.1, TXLED.A; no longer C6.1, IC3.3, R1.2, R2.1
- net N$3: now also ONLED.A, R8.1; no longer R18.1, T1.B
- net PAD1: now also C29.2, PAD1A.1, PAD1B.P$1, PAD1B.P$2, R21.2; no longer R24.1
- net PAD2: now also C31.2, PAD2A.1, PAD2B.P$1, PAD2B.P$2, R22.2; no longer R23.1
- net PAD3: now also C25.2, PAD3A.1, PAD3B.P$1, PAD3B.P$2, R19.2; no longer R25.1
- net PAD4: now also C27.2, PAD4A.1, PAD4B.P$1, PAD4B.P$2, R20.2; no longer R26.1
- net RESET: now also D1.A, JP1.5, R1.1; no longer D2.A, JP1.6, JP3.5, R3.1, U2.13
- net RXLED: now also RXLED.C; no longer R11.2, U2.8
- net SCK: now also JP1.3; no longer JP3.3, U2.9
- net TXLED: now also TXLED.C; no longer R10.1, U2.22
- net VBAT: now also IC5.14, U$1.+$1, U$1.+$2; no longer G1.+, IC4.14
- net VCC: now also C32.+, C33.+, C34.1, LED1.1-VDD, LED10.1-VDD, LED100.1-VDD, LED101.1-VDD, LED102.1-VDD, LED103.1-VDD, LED104.1-VDD, LED105.1-VDD, LED106.1-VDD, LED107.1-VDD, LED108.1-VDD, LED109.1-VDD, LED11.1-VDD, LED110.1-VDD, LED111.1-VDD, LED112.1-VDD, LED113.1-VDD, LED114.1-VDD, LED115.1-VDD, LED116.1-VDD, LED117.1-VDD, LED118.1-VDD, LED119.1-VDD, LED12.1-VDD, LED120.1-VDD, LED121.1-VDD, LED122.1-VDD, LED123.1-VDD, LED124.1-VDD, LED125.1-VDD, LED126.1-VDD, LED127.1-VDD, LED128.1-VDD, LED129.1-VDD, LED13.1-VDD, LED130.1-VDD, LED131.1-VDD, LED132.1-VDD, LED133.1-VDD, LED134.1-VDD, LED135.1-VDD, LED136.1-VDD, LED137.1-VDD, LED138.1-VDD, LED139.1-VDD, LED14.1-VDD, LED140.1-VDD, LED141.1-VDD, LED142.1-VDD, LED143.1-VDD, LED144.1-VDD, LED15.1-VDD, LED16.1-VDD, LED17.1-VDD, LED18.1-VDD, LED19.1-VDD, LED2.1-VDD, LED20.1-VDD, LED21.1-VDD, LED22.1-VDD, LED23.1-VDD, LED24.1-VDD, LED25.1-VDD, LED26.1-VDD, LED27.1-VDD, LED28.1-VDD, LED29.1-VDD, LED3.1-VDD, LED30.1-VDD, LED31.1-VDD, LED32.1-VDD, LED33.1-VDD, LED34.1-VDD, LED35.1-VDD, LED36.1-VDD, LED37.1-VDD, LED38.1-VDD, LED39.1-VDD, LED4.1-VDD, LED40.1-VDD, LED41.1-VDD, LED42.1-VDD, LED43.1-VDD, LED44.1-VDD, LED45.1-VDD, LED46.1-VDD, LED47.1-VDD, LED48.1-VDD, LED49.1-VDD, LED5.1-VDD, LED50.1-VDD, LED51.1-VDD, LED52.1-VDD, LED53.1-VDD, LED54.1-VDD, LED55.1-VDD, LED56.1-VDD, LED57.1-VDD, LED58.1-VDD, LED59.1-VDD, LED6.1-VDD, LED60.1-VDD, LED61.1-VDD, LED62.1-VDD, LED63.1-VDD, LED64.1-VDD, LED65.1-VDD, LED66.1-VDD, LED67.1-VDD, LED68.1-VDD, LED69.1-VDD, LED7.1-VDD, LED70.1-VDD, LED71.1-VDD, LED72.1-VDD, LED73.1-VDD, LED74.1-VDD, LED75.1-VDD, LED76.1-VDD, LED77.1-VDD, LED78.1-VDD, LED79.1-VDD, LED8.1-VDD, LED80.1-VDD, LED81.1-VDD, LED82.1-VDD, LED83.1-VDD, LED84.1-VDD, LED85.1-VDD, LED86.1-VDD, LED87.1-VDD, LED88.1-VDD, LED89.1-VDD, LED9.1-VDD, LED90.1-VDD, LED91.1-VDD, LED92.1-VDD, LED93.1-VDD, LED94.1-VDD, LED95.1-VDD, LED96.1-VDD, LED97.1-VDD, LED98.1-VDD, LED99.1-VDD, U4.2; no longer C16.1, C7.1, C8.1, D2.C, I1.1, IC1.3, Q1.2, R3.2, U1.14, U1.2, U1.24, U1.34, U2.14, U2.2, U2.24, U2.34
- net VIN: now also C9.+, CN2.VBUS, D5.C, IC1.3, JP2.POWER, R11.2, U4.1; no longer C1.1, D1.C, IC1.1, IC5.1, JP4.1, R1.1, U$2.VBUS
- net VUSB: now also C10.+, C11.2, I1.1, T1.1; no longer C12.1, C13.1, F1.1, Q1.3, U2.7
- net XTAL1: now also C7.1, R2.1, Y1.1; no longer C14.2, R8.2, U2.17, Y1.2
- net XTAL2: now also C5.2, R2.2, Y1.2; no longer C15.2, R8.1, U2.16, Y1.1
Routing:
- net VCC: track 0.00 -> 3849.0 mm, vias 0 -> 1
- net +5V: track 0.00 -> 1193.1 mm, vias 0 -> 14
- net IO11*: track 0.00 -> 268.7 mm, vias 0 -> 4
- net N$146: track 0.00 -> 263.5 mm
- net N$145: track 0.00 -> 263.5 mm
- net N$144: track 0.00 -> 263.5 mm
- net N$143: track 0.00 -> 263.5 mm
- net N$142: track 0.00 -> 263.5 mm
- net N$141: track 0.00 -> 263.5 mm
- net N$140: track 0.00 -> 263.5 mm
- net N$139: track 0.00 -> 263.5 mm
- net N$138: track 0.00 -> 263.5 mm
- net N$137: track 0.00 -> 263.5 mm
- net N$136: track 0.00 -> 263.5 mm
- net A4: track 0.00 -> 242.3 mm, vias 0 -> 2
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Other:
- board size 240 x 240 mm -> 300 x 300 mm
- board text added: "X2"

Commit message: V1.3 PCB
Parts:
- removed CN1, CN2: (no value), adafruit:USB-MINIB-THM
- removed D6: BLUE, SparkFun-LED:LED-1206
- removed J1, J2, J3, J4: 22-05-7028-02, con-molex:7395-02
- removed S10, S11, S12, S9: SWITCH-MOMENTARY-2TACTILE-SWITCH-SMD-RIGHT-ANGLE, SparkFun-Electromechanical:TACTILE_SWITCH-SMD-RIGHT-ANGLE
- removed U$2, U$3, U$4, U$5: AT42QT1010SOT23, SparkFun-DigitalIC:SOT23-6
- removed X1: (no value), adafruit:ESP-12
- added +5VDC: POWER_JACKPTH, SparkFun-Connectors:POWER_JACK_PTH
- added CR1: CR2032, adafruit:CR2032-SMD
- added D2: CD1206-S01575, diode:MINIMELF
- added DATA: USBDATA, adafruit:USB-MINIB-THM-MOLEX
- added ESP12: ESP12, adafruit:ESP-12
- added IC7: LMV358IDGKR, linear:SO08
- added ICSP: ICSP, pinhead:2X03/90
- added JP3, JP4: (no value), pinhead:1X02/90
- added POWER: USBPOWER, adafruit:USB-MINIB-THM-MOLEX
- added RESET, SW10, SW11: SWITCH-MOMENTARY-2SMD-1101NE, SparkFun-Electromechanical:TACTILE-SWITCH-1101NE
- added S4: JS202011SCQN, switch-ck:JS202011SCQN
- added U2: HC_05, SerialPortBluetooth:BLUETOOTH_SMD
- added U5: NCP1117ST50T3G, linear:SOT223
- added U6: LP2985-33DBVR, SmartPrj:SOT23-DBV
- BLUETOOTH, DS3231: value (none) -> SSM-106-S-SH; device SparkFun-Connectors:1X06-SMD-FEMALE-V2 -> SAMTEC-FLE-Mxx-Sxx_By_element14_Batch_1:SAMTEC_SSM-106-S-SH
- C1: value 100n -> 1uF; device resistor:C1206 -> resistor:B/3528-21W
- C10, C9: value 10u -> 22p; device resistor:SMC_C -> resistor:C1206
- C11, C22, C31: value 100n -> 1u; device resistor:C1206 -> resistor:B/3528-21W
- C13, C15: value 1u -> 100n; device resistor:SMC_C -> resistor:C1206
- C16, C17, C20: value 1u -> 100n; device resistor:SMC_A -> resistor:C1206
- C21: device resistor:SMC_A -> resistor:B/3528-21W
- C27, C28, C29, C30, C34: value 100n -> 10u; device resistor:C1206 -> resistor:B/3528-21W
- C3: device resistor:SMC_C -> resistor:B/3528-21W
- C32: value 10u -> 1u; device resistor:SMC_C -> resistor:B/3528-21W
- C33, C8: value 10u -> 100n; device resistor:SMC_C -> resistor:C1206
- C4: value 1uF -> 100n; device resistor:SMC_C -> resistor:C1206
- C5: value 22p -> 100n
- C7: value 22p -> 1u; device resistor:C1206 -> resistor:B/3528-21W
- D1: value CD1206-S01575 -> BLUE; device diode:MINIMELF -> SparkFun-LED:LED-1206
- H1, H2, H3, H4: value MOUNT-HOLE5.5 -> (none); device holes:5,5 -> holes:2,8-PAD
- IC1: value NCP1117ST50T3G -> ATMEGA32U4TQFP-44; device linear:SOT223 -> SparkFun-DigitalIC:TQFP44
- IC2: value LMV358IDGKR -> DS3231/SO; device linear:SO08 -> adafruit:SO16W
- IC3, IC4, IC6: value LP2985-33DBVR -> AT42QT1010SOT23; device SmartPrj:SOT23-DBV -> SparkFun-DigitalIC:SOT23-6
- IC5: value DS3231/SO -> AT42QT1010SOT23; device adafruit:SO16W -> SparkFun-DigitalIC:SOT23-6
- JP1: device pinhead:2X03/90 -> pinhead:1X02/90
- JP2: value POWER_JACKCOMBO -> (none); device SparkFun-Connectors:POWER_JACK_COMBO -> pinhead:1X02/90
- PAD1A: value (none) -> PAD1A
- PAD1B, PAD2B, PAD3B, PAD4B: device SparkFun-Electromechanical:CAPSENSE_PAD -> David:CAPSENSE_PAD
- PAD2A: value (none) -> PAD2A
- PAD3A: value (none) -> PAD3A
- PAD4A: value (none) -> PAD4A
- R1, R12: value 10K -> 1K
- R10: value 22R -> 1M
- R11, R3: value 10K -> 12K
- R13: value 470 -> 22K
- R15, R17, R18: value 22K -> 12K
- R19, R20: value 12K -> 22K
- R2: value 1M -> 12K
- R21, R22: value 12K -> 10K
- R23: value PHOTOCELLPTH -> K; device SparkFun-Sensors:PHOTOCELL -> resistor:R1206
- R24: value PHOTOCELLPTH -> 22R; device SparkFun-Sensors:PHOTOCELL -> resistor:R1206
- R25: value 12K -> 22R
- R26, R27, R28: value 12K -> PHOTOCELLPTH; device resistor:R1206 -> SparkFun-Sensors:PHOTOCELL
- R29: value 470 -> PHOTOCELLPTH; device resistor:R1206 -> SparkFun-Sensors:PHOTOCELL
- R4, R5: value PHOTOCELLPTH -> 12K; device SparkFun-Sensors:PHOTOCELL -> resistor:R1206
- R6, R7: value 1K -> 470
- R8: value K -> 10K
- R9: value 22R -> 10K
- S1, S2, S3: value SWITCH-MOMENTARY-2SMD-1101NE -> JS202011SCQN; device SparkFun-Electromechanical:TACTILE-SWITCH-1101NE -> switch-ck:JS202011SCQN
- S5, S6, S7, S8: device SparkFun-Electromechanical:AYZ0202 -> switch-omron:B3F-31XX
- U$1: device adafruit:CR2032-SMD -> David:FIREBIRD2
- U1: value ATMEGA32U4TQFP-44 -> LP2985-33DBVR; device SparkFun-DigitalIC:TQFP44 -> SmartPrj:SOT23-DBV
- U3: value HC_05 -> LP2985-33DBVR; device SerialPortBluetooth:BLUETOOTH_SMD -> SmartPrj:SOT23-DBV
- moved H3 381.8 mm to (290.0, 290.0)
- moved S8 285.7 mm to (296.5, 79.0), flipped to the bottom, turned to 270 degrees
- moved R24 278.3 mm to (193.0, 22.0), flipped to the top, turned to 90 degrees
- moved H1 270.2 mm to (10.0, 10.0)
- moved H2 270.2 mm to (10.0, 290.0)
- moved S5 209.7 mm to (296.5, 112.0), flipped to the bottom, turned to 270 degrees
- moved R27 197.3 mm to (20.0, 240.0), flipped to the bottom, turned to 0 degrees
- moved C28 182.3 mm to (107.0, 22.0), turned to 90 degrees
- moved R4 178.5 mm to (168.0, 101.0), flipped to the top, turned to 90 degrees
- moved PAD2A 178.3 mm to (185.0, 17.0), flipped to the bottom, turned to 180 degrees
- moved PAD2B 178.0 mm to (185.0, 8.00)
- moved R26 176.0 mm to (280.0, 240.0), flipped to the bottom, turned to 0 degrees
- moved C29 160.0 mm to (130.0, 22.0), turned to 90 degrees
- moved R21 157.1 mm to (139.0, 30.5), turned to 90 degrees
- moved PAD4A 153.3 mm to (45.0, 17.0), flipped to the bottom, turned to 180 degrees
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- renumbered D5 to D3
Connections:
- removed net USBID: CN1.ID
- net +3V3: now also C32.+, IC7.6, U6.5; no longer C13.-, IC2.6, IC3.5
- net +3V3B: now also C6.2, C7.+, U1.5, U2.12; no longer C17.-, C19.2, IC4.5, U3.12
- net +3V3C: now also C22.+, ESP12.8, R19.1, U3.5; no longer C21.-, IC6.5, R18.2, X1.8
- net +5V: now also C11.+, C20.1, C21.+, C25.2, C30.+, C31.+, C4.1, C5.1, C8.2, D2.C, IC1.14, IC1.34, IC2.2, IC3.5, IC4.5, IC5.5, IC6.5, IC7.8, ICSP.2, R1.1, R12.2, R23.1, R26.2, R27.2, R28.2, R29.2, R8.1, S1.6, S2.6, S3.6, S4.6, U1.1, U1.3, U3.1, U3.3, U5.2, U5.4, U6.1, U6.3; no longer C1.1, C12.1, C15.-, C16.-, C18.2, C2.1, C20.-, C22.2, C8.+, D1.C, IC1.4, IC2.8, IC3.1, IC3.3, IC4.1, IC4.3, IC5.2, IC6.1, IC6.3, JP1.2, R1.2, R23.2, R24.2, R4.2, R5.2, R6.2, R7.2, R8.2, S5.1, S6.1, S7.1, S8.1, U$2.5, U$3.5, U$4.5, U$5.5, U1.14, U1.2, U1.34
- net A0: now also IC1.36, JP2.1, S6.1; no longer J3.1, S10.1, U1.36
- net A1: now also IC1.37, JP1.1, S5.1; no longer J4.1, S9.1, U1.37
- net A2: now also IC1.38, R28.1; no longer R26.2, U1.38
- net A3: now also IC1.39, R26.1; no longer R25.2, U1.39
- net A4: now also IC1.40, R27.1, R3.1; no longer R24.1, R28.2, U1.40
- net A5: now also IC1.41, R2.1, R29.1; no longer R23.1, R27.2, U1.41
- net AREF: now also C2.1, IC1.42; no longer C6.2, U1.42
- net AVCC: now also C1.+, IC1.24, IC1.44; no longer C3.+, U1.24, U1.44
- net BLUETOOTHLED: now also D1.A, R7.2; no longer D6.A, R13.2
- net CMP: now also C24.2, IC7.5, R21.2, R22.2; no longer C14.2, IC2.5, R11.1, R12.2
- net D+: now also DATA.D+, R24.1; no longer CN1.D+, R9.1
- net D-: now also DATA.D-, R25.1; no longer CN1.D-, R10.1
- net D0/RX: now also ESP12.16, IC1.20; no longer U1.20, X1.16
- net D1/TX: now also IC1.21, R14.1, R20.2; no longer R16.1, R17.1, U1.21
- net D2/SDA: now also IC1.19, IC2.15; no longer IC5.15, U1.19
- net D3/SCL: now also IC1.18, IC2.16; no longer IC5.16, U1.18
- net D4: now also IC1.25, IC3.1; no longer U$5.1, U1.25
- net D5*: now also IC1.31, JP4.1, S8.1; no longer J1.1, S12.1, U1.31
- net D6*: now also IC1.27, IC5.1; no longer U$3.1, U1.27
- net D7: now also IC1.1, R6.1; no longer R29.1, U1.1
- net DS3231RST: now also IC2.4, SW10.2; no longer IC5.4, S3.2
- net ESP12RESET: now also ESP12.1, R19.2, SW11.2; no longer R18.1, S2.2, X1.1
- net ESP12RX: now also ESP12.15, R14.2; no longer R16.2, X1.15
- net GATE_CMD: now also IC7.7; no longer IC2.7
- net GND: now also +5VDC.GND, +5VDC.GNDBREAK, C1.-, C10.1, C11.-, C14.2, C16.2, C18.2, C20.2, C21.-, C22.-, C24.1, C26.1, C27.-, C28.-, C29.-, C30.-, C31.-, C33.1, C34.-, C4.2, C5.2, C7.-, C8.1, C9.2, CR1.-, D1.C, DATA.GND, ESP12.9, H1.B2,8, H2.B2,8, H3.B2,8, H4.B2,8, IC1.15, IC1.23, IC1.35, IC1.43, IC1.5, IC2.10, IC2.11, IC2.12, IC2.13, IC2.5, IC2.6, IC2.7, IC2.8, IC2.9, IC5.2, IC7.4, ICSP.6, JP1.2, JP2.2, JP3.2, JP4.2, POWER.GND, R13.2, R2.2, R20.1, R22.1, R4.2, R5.2, R9.2, RESET.2, S1.1, S1.4, S2.4, S3.4, S4.1, S4.4, S5.2, S6.2, S7.2, S8.2, SW10.1, SW11.1, U1.2, U2.13, U2.21, U2.22, U3.2, U5.1, U6.2; no longer C1.2, C10.-, C11.1, C13.+, C14.1, C15.+, C16.+, C17.+, C18.1, C19.1, C20.+, C21.+, C22.1, C27.1, C29.1, C31.1, C33.-, C34.2, C4.-, C5.1, C7.2, C8.-, C9.-, CN1.GND, CN2.GND, D6.C, IC1.1, IC2.4, IC5.10, IC5.11, IC5.12, IC5.13, IC5.5, IC5.6, IC5.7, IC5.8, IC5.9, J1.2, J2.2, J3.2, J4.2, JP1.6, JP2.GND, JP2.GND@1, R12.1, R15.1, R17.2, R25.1, R26.1, R27.1, R28.1, S1.2, S10.2, S11.2, S12.2, S5.3, S6.3, S7.3, S8.3, S9.2, U$1.-, U$2.2, U$3.2, U$4.2, U$5.2, U1.15, U1.23, U1.35, U1.43, U1.5, U3.13, U3.21, U3.22, X1.9
- net HC-05RX: now also R11.2, U2.2; no longer R14.2, U3.2
- net HWB: now also IC1.33, R9.1; no longer R3.1, U1.33
- net IO10*: now also IC1.30, U2.1; no longer U1.30, U3.1
- net IO11*: now also IC1.12, R11.1, R13.1; no longer R14.1, R15.2, U1.12
- net IO12: now also IC1.26, IC4.1; no longer U$2.1, U1.26
- net IO13*: now also IC1.32, JP3.1, S7.1; no longer J2.1, S11.1, U1.32
- net IO8: now also IC1.28, IC6.1; no longer U$4.1, U1.28
- net IO9*: now also IC1.29, U2.34; no longer U1.29, U3.34
- net MISO: now also IC1.11, ICSP.1; no longer JP1.1, U1.11
- net MODE1: now also IC6.6, S1.5; no longer S7.2, U$4.6
- net MODE2: now also IC3.6, S2.5; no longer S8.2, U$5.6
- net MODE3: now also IC4.6, S3.5; no longer S5.2, U$2.6
- net MODE4: now also IC5.6, S4.5; no longer S6.2, U$3.6
- net MOSI: now also IC1.10, ICSP.4; no longer JP1.4, U1.10
- net N$1: now also R12.1; no longer R6.1
- net N$147: now also R6.2; no longer R29.2
- net N$2: now also R1.2; no longer R7.1
- net N$3: now also R23.2; no longer R8.1
- net PAD1: now also C18.1, R18.1; no longer C29.2, PAD1B.P$2, R21.2
- net PAD2: now also C16.1, R17.1; no longer C31.2, PAD2B.P$2, R22.2
- net PAD3: now also C14.1, R16.1; no longer C25.2, PAD3B.P$2, R19.2
- net PAD4: now also C12.1, R15.1; no longer C27.2, PAD4B.P$2, R20.2
- net RD+: now also IC1.4, R24.2; no longer R9.2, U1.4
- net RD-: now also IC1.3, R25.2; no longer R10.2, U1.3
- net RESET: now also D2.A, IC1.13, ICSP.5, R8.2, RESET.1; no longer D1.A, JP1.5, R1.1, S1.1, U1.13
- net RXLED: now also IC1.8; no longer U1.8
- net SCK: now also IC1.9, ICSP.3; no longer JP1.3, U1.9
- net SNS1: now also C19.2, IC6.4; no longer C28.1, U$4.4
- net SNS2: now also C13.2, IC3.4; no longer C30.1, U$5.4
- net SNS3: now also C15.2, IC4.4; no longer C24.1, U$2.4
- net SNS4: now also C17.2, IC5.4; no longer C26.1, U$3.4
- net SNSK1: now also C19.1, IC6.3, R18.2; no longer C28.2, R21.1, U$4.3
- net SNSK2: now also C13.1, IC3.3, R15.2; no longer C30.2, R22.1, U$5.3
- net SNSK3: now also C15.1, IC4.3, R16.2; no longer C24.2, R19.1, U$2.3
- net SNSK4: now also C17.1, IC5.3, R17.2; no longer C26.2, R20.1, U$3.3
- net STATE: now also R7.1, U2.31; no longer R13.1, U3.31
- net TXLED: now also IC1.22; no longer U1.22
- net UCAP: now also C3.+, IC1.6; no longer C4.+, U1.6
- net VBAT: now also CR1.+$1, CR1.+$2, IC2.14; no longer IC5.14, U$1.+$1, U$1.+$2
- net VCC: now also C26.2, C27.+, C28.+; no longer C32.+, C33.+, C34.1
- net VIN: now also +5VDC.PWR, C29.+, POWER.VBUS, R21.1, U5.3; no longer C9.+, CN2.VBUS, IC1.3, JP2.POWER, R11.2
- net VUSB: now also C33.2, C34.+, I1.2, IC1.7; no longer C10.+, C11.2, I1.1, U1.7
- net XTAL1: now also C10.2, IC1.17, R10.1, Y1.2; no longer C7.1, R2.1, U1.17, Y1.1
- net XTAL2: now also C9.1, IC1.16, R10.2, Y1.1; no longer C5.2, R2.2, U1.16, Y1.2
- net XUSB: now also DATA.VBUS, I1.1; no longer CN1.VBUS, I1.2
Routing:
- net D4: track 211.0 -> 27.3 mm, vias 8 -> 0
- net PAD4: track 12.6 -> 172.3 mm, vias 0 -> 1
- net IO8: track 172.0 -> 48.6 mm
- net PAD1: track 11.4 -> 112.7 mm, vias 0 -> 2
- net PAD3: track 8.01 -> 101.4 mm, vias 0 -> 1
- net D6*: track 126.8 -> 37.8 mm
- net IO11*: track 268.7 -> 183.9 mm, vias 4 -> 5
- net IO12: track 113.9 -> 29.6 mm, vias 4 -> 0
- net VIN: track 66.5 -> 119.8 mm
- net PAD2: track 0.00 -> 52.9 mm, vias 0 -> 1
- net +5V: track 1193.1 -> 1149.9 mm, vias 14 -> 11
- net VBAT: track 76.9 -> 43.1 mm
- net D3/SCL: track 77.8 -> 102.2 mm, vias 4 -> 2
- net GND: track 0.00 -> 22.5 mm, vias 0 -> 19
- net D-: track 58.2 -> 39.9 mm
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- added copper zone on layer 1, net GND
- added copper zone on layer 16, net GND
Other:
- board text added: "+5V DC"
- board text added: "3A"
- board text added: "ATMEGA32U4"
- board text added: "DS3231 RTC MODULE"
- board text added: "EXTERNAL SWITCH HEADERS"
- board text added: "HC-05 BLUETOOTH MODULE"
- board text added: "PAD1A"
- board text added: "PAD2A"
- board text added: "PAD3A"
- board text added: "PAD4A"
- board text added: "SIDE MOUNTED SWITCHES"
- board text removed: "X2"
