File: Eagle/Word-Clock.sch (EAGLE design)
At the start: 267 parts, among them IC1 NCP1117ST50T3G, IC2 LMV358IDGKR, IC3 LP2985-33DBVR, IC4 LP2985-33DBVR, IC5 DS3231/SO, IC6 LP2985-33DBVR, J1 22-05-7028-02, J2 22-05-7028-02, J3 22-05-7028-02, J4 22-05-7028-02, T1 FDN340P, U1 ATMEGA32U4TQFP-44, U3 HC_05, U4 +12v, Y1 16MHz

Commit message: V1.3 PCB
Parts:
- removed CN1, CN2: (no value), adafruit:USBTHM
- removed D5: M7, diode:DIODE-SMB
- removed D6: BLUE, SparkFun-LED:LED-BLUE1206
- removed J1, J2, J3, J4: 22-05-7028-02, con-molex:22-05-7028-02
- removed S10, S11, S12, S9: SWITCH-MOMENTARY-2TACTILE-SWITCH-SMD-RIGHT-ANGLE, SparkFun-Electromechanical:SWITCH-MOMENTARY-2TACTILE-SWITCH-SMD-RIGHT-ANGLE
- removed U$2, U$3, U$4, U$5: AT42QT1010SOT23, SparkFun-DigitalIC:AT42QT1010SOT23
- added +5VDC: POWER_JACKPTH, SparkFun-Connectors:POWER_JACKPTH
- added D2: CD1206-S01575, diode:DIODE-MINIMELF
- added D3: M7, diode:DIODE-SMB
- added DATA: USBDATA, adafruit:USBMOLEX
- added IC7: LMV358IDGKR, linear:LMV358MX
- added ICSP: ICSP, pinhead:PINHD-2X3/90
- added JP3, JP4: (no value), pinhead:PINHD-1X2/90
- added POWER: USBPOWER, adafruit:USBMOLEX
- added RESET, SW10, SW11: SWITCH-MOMENTARY-2SMD-1101NE, SparkFun-Electromechanical:SWITCH-MOMENTARY-2SMD-1101NE
- added S4: JS202011SCQN, switch-ck:JS202011SCQN
- added U2: HC_05, SerialPortBluetooth:HC_05
- added U5: NCP1117ST50T3G, linear:MC33269ST-3.3T3
- added U6: LP2985-33DBVR, SmartPrj:LP2985-XXDBVR33
- BLUETOOTH, DS3231: value (none) -> SSM-106-S-SH; device SparkFun-Connectors:M06SMD-FEMALE-V2 -> SAMTEC-FLE-Mxx-Sxx_By_element14_Batch_1:SSM-106-S-SH
- C1: value 100n -> 1uF; device resistor:C-EUC1206 -> resistor:CPOL-EUB/3528-21W
- C10, C9: value 10u -> 22p; device resistor:CPOL-EUSMCC -> resistor:C-EUC1206
- C11, C22, C31: value 100n -> 1u; device resistor:C-EUC1206 -> resistor:CPOL-EUB/3528-21W
- C13, C15: value 1u -> 100n; device resistor:CPOL-EUSMCC -> resistor:C-EUC1206
- C16, C17, C20: value 1u -> 100n; device resistor:CPOL-EUSMCA -> resistor:C-EUC1206
- C21: device resistor:CPOL-EUSMCA -> resistor:CPOL-EUB/3528-21W
- C27, C28, C29, C30, C34: value 100n -> 10u; device resistor:C-EUC1206 -> resistor:CPOL-EUB/3528-21W
- C3: device resistor:CPOL-EUSMCC -> resistor:CPOL-EUB/3528-21W
- C32: value 10u -> 1u; device resistor:CPOL-EUSMCC -> resistor:CPOL-EUB/3528-21W
- C33, C8: value 10u -> 100n; device resistor:CPOL-EUSMCC -> resistor:C-EUC1206
- C4: value 1uF -> 100n; device resistor:CPOL-EUSMCC -> resistor:C-EUC1206
- C5: value 22p -> 100n
- C7: value 22p -> 1u; device resistor:C-EUC1206 -> resistor:CPOL-EUB/3528-21W
- CR1: value (none) -> CR2032
- D1: value CD1206-S01575 -> BLUE; device diode:DIODE-MINIMELF -> SparkFun-LED:LED-BLUE1206
- ESP12: value (none) -> ESP12
- H1, H2, H3, H4: value MOUNT-HOLE5.5 -> MOUNT-PAD-ROUND2.8; device holes:MOUNT-HOLE5.5 -> holes:MOUNT-PAD-ROUND2.8
- IC1: value NCP1117ST50T3G -> ATMEGA32U4TQFP-44; device linear:MC33269ST-3.3T3 -> SparkFun-DigitalIC:ATMEGA32U4TQFP-44
- IC2: value LMV358IDGKR -> DS3231/SO; device linear:LMV358MX -> adafruit:DS3231/SO
- IC3, IC4, IC6: value LP2985-33DBVR -> AT42QT1010SOT23; device SmartPrj:LP2985-XXDBVR33 -> SparkFun-DigitalIC:AT42QT1010SOT23
- IC5: value DS3231/SO -> AT42QT1010SOT23; device adafruit:DS3231/SO -> SparkFun-DigitalIC:AT42QT1010SOT23
- JP1: device pinhead:PINHD-2X3/90 -> pinhead:PINHD-1X2/90
- JP2: value POWER_JACKCOMBO -> (none); device SparkFun-Connectors:POWER_JACKCOMBO -> pinhead:PINHD-1X2/90
- ONLED: FARNELL (none) -> 2322084
- PAD1A: value (none) -> PAD1A
- PAD1B, PAD2B, PAD3B, PAD4B: device SparkFun-Electromechanical:CAPSENSE_PAD -> David:CAPSENSE_PAD
- PAD2A: value (none) -> PAD2A
- PAD3A: value (none) -> PAD3A
- PAD4A: value (none) -> PAD4A
- R1, R12: value 10K -> 1K
- R10: value 22R -> 1M
- R11, R3: value 10K -> 12K
- R13: value 470 -> 22K
- R15, R17, R18: value 22K -> 12K
- R19, R20: value 12K -> 22K
- R2: value 1M -> 12K
- R21, R22: value 12K -> 10K
- R23: value PHOTOCELLPTH -> K; device SparkFun-Sensors:PHOTOCELLPTH -> resistor:R-EU_R1206
- R24: value PHOTOCELLPTH -> 22R; device SparkFun-Sensors:PHOTOCELLPTH -> resistor:R-EU_R1206
- R25: value 12K -> 22R
- R26, R27, R28: value 12K -> PHOTOCELLPTH; device resistor:R-EU_R1206 -> SparkFun-Sensors:PHOTOCELLPTH
- R29: value 470 -> PHOTOCELLPTH; device resistor:R-EU_R1206 -> SparkFun-Sensors:PHOTOCELLPTH
- R4, R5: value PHOTOCELLPTH -> 12K; device SparkFun-Sensors:PHOTOCELLPTH -> resistor:R-EU_R1206
- R6, R7: value 1K -> 470
- R8: value K -> 10K
- R9: value 22R -> 10K
- RXLED: FARNELL (none) -> 2322085
- S1, S2, S3: value SWITCH-MOMENTARY-2SMD-1101NE -> JS202011SCQN; device SparkFun-Electromechanical:SWITCH-MOMENTARY-2SMD-1101NE -> switch-ck:JS202011SCQN; PROD_ID 1703878 -> (none)
- S5, S6, S7, S8: device SparkFun-Electromechanical:SWITCH-SPDTSMD -> switch-omron:31-XX
- U1: value ATMEGA32U4TQFP-44 -> LP2985-33DBVR; device SparkFun-DigitalIC:ATMEGA32U4TQFP-44 -> SmartPrj:LP2985-XXDBVR33
- U3: value HC_05 -> LP2985-33DBVR; device SerialPortBluetooth:HC_05 -> SmartPrj:LP2985-XXDBVR33
- renumbered U$1 to CR1, X1 to ESP12
Connections:
- removed net USBID: CN1.ID
- net +3V3: now also C32.+, IC7B.-IN, U6.OUT; no longer C13.-, IC2B.-IN, IC3.OUT
- net +3V3B: now also C6.2, C7.+, U1.OUT, U2.3V3; no longer C17.-, C19.2, IC4.OUT, U3.3V3
- net +3V3C: now also C22.+, R19.1, U3.OUT; no longer C21.-, IC6.OUT, R18.2
- net +5V: now also C11.+, C20.1, C21.+, C25.2, C30.+, C31.+, C4.1, C5.1, C8.2, D2.C, IC1.UVCC, IC1.VCC@14, IC1.VCC@34, IC2.VCC, IC3.VDD, IC4.VDD, IC5.VDD, IC6.VDD, IC7P.V+, ICSP.2, R1.1, R12.2, R23.1, R26.P$2, R27.P$2, R28.P$2, R29.P$2, R8.1, S1.6, S2.6, S3.6, S4.6, U1.IN, U1.ON/!OFF, U3.IN, U3.ON/!OFF, U5.OUT, U5.OUT@1, U6.IN, U6.ON/!OFF; no longer C1.1, C12.1, C15.-, C16.-, C18.2, C2.1, C20.-, C22.2, C8.+, D1.C, IC1.OUT, IC1.OUT@1, IC2P.V+, IC3.IN, IC3.ON/!OFF, IC4.IN, IC4.ON/!OFF, IC5.VCC, IC6.IN, IC6.ON/!OFF, JP1.2, R1.2, R23.P$2, R24.P$2, R4.P$2, R5.P$2, R6.2, R7.2, R8.2, S5.O, S6.O, S7.O, S8.O, U$2.VDD, U$3.VDD, U$4.VDD, U$5.VDD, U1.UVCC, U1.VCC@14, U1.VCC@34
- net A0: now also IC1.PF7(ADC7), JP2.1, S6.P; no longer J3-1.S, S10.1, U1.PF7(ADC7)
- net A1: now also IC1.PF6(ADC6), JP1.1, S5.P; no longer J4-1.S, S9.1, U1.PF6(ADC6)
- net A2: now also IC1.PF5(ADC5), R28.P$1, R5.1; no longer R26.2, R5.P$1, U1.PF5(ADC5)
- net A3: now also IC1.PF4(ADC4), R26.P$1, R4.1; no longer R25.2, R4.P$1, U1.PF4(ADC4)
- net A4: now also IC1.PF1(ADC1), R27.P$1, R3.1; no longer R24.P$1, R28.2, U1.PF1(ADC1)
- net A5: now also IC1.PF0(ADC0), R2.1, R29.P$1; no longer R23.P$1, R27.2, U1.PF0(ADC0)
- net AREF: now also C2.1, IC1.AREF; no longer C6.2, U1.AREF
- net AVCC: now also C1.+, IC1.AVCC@24, IC1.AVCC@44; no longer C3.+, U1.AVCC@24, U1.AVCC@44
- net BLUETOOTHLED: now also D1.A, R7.2; no longer D6.A, R13.2
- net CMP: now also C24.2, IC7B.+IN, R21.2, R22.2; no longer C14.2, IC2B.+IN, R11.1, R12.2
- net D+: now also DATA.D+, R24.1; no longer CN1.D+, R9.1
- net D-: now also DATA.D-, R25.1; no longer CN1.D-, R10.1
- net D0/RX: now also IC1.PD2(RX); no longer U1.PD2(RX)
- net D1/TX: now also IC1.PD3(TX), R14.1, R20.2; no longer R16.1, R17.1, U1.PD3(TX)
- net D2/SDA: now also IC1.PD1(SDA), IC2.SDA; no longer IC5.SDA, U1.PD1(SDA)
- net D3/SCL: now also IC1.PD0(SCL), IC2.SCL; no longer IC5.SCL, U1.PD0(SCL)
- net D4: now also IC1.PD4(ADC8), IC3.OUT; no longer U$5.OUT, U1.PD4(ADC8)
- net D5*: now also IC1.PC6, JP4.1, S8.P; no longer J1-1.S, S12.1, U1.PC6
- net D6*: now also IC1.PD7(ADC10), IC5.OUT; no longer U$3.OUT, U1.PD7(ADC10)
- net D7: now also IC1.PE6, R6.1; no longer R29.1, U1.PE6
- net DS3231RST: now also IC2./RST, SW10.2; no longer IC5./RST, S3.2
- net ESP12RESET: now also R19.2, SW11.2; no longer R18.1, S2.2
- net ESP12RX: now also R14.2; no longer R16.2
- net GATE_CMD: now also IC7B.OUT; no longer IC2B.OUT
- net GND: now also +5VDC.GND, +5VDC.GNDBREAK, C1.-, C10.1, C11.-, C14.2, C16.2, C18.2, C20.2, C21.-, C22.-, C24.1, C26.1, C27.-, C28.-, C29.-, C30.-, C31.-, C33.1, C34.-, C4.2, C5.2, C7.-, C8.1, C9.2, D1.C, D3.A, DATA.GND, H1.MOUNT, H2.MOUNT, H3.MOUNT, H4.MOUNT, IC1.GND@15, IC1.GND@23, IC1.GND@35, IC1.GND@43, IC1.UGND, IC2.GND, IC2.NC, IC2.NC1, IC2.NC2, IC2.NC3, IC2.NC4, IC2.NC5, IC2.NC6, IC2.NC7, IC3.VSS, IC4.VSS, IC5.VSS, IC6.VSS, IC7P.V-, ICSP.6, JP1.2, JP2.2, JP3.2, JP4.2, POWER.GND, R13.2, R2.2, R20.1, R22.1, R4.2, R5.2, R9.2, RESET.2, S1.1, S1.4, S2.4, S3.4, S4.1, S4.4, SW10.1, SW11.1, U1.GND, U2.GND, U2.GND1, U2.GND2, U5.GND/ADJ, U6.GND; no longer C1.2, C10.-, C11.1, C13.+, C14.1, C15.+, C16.+, C17.+, C18.1, C19.1, C20.+, C21.+, C22.1, C27.1, C29.1, C31.1, C33.-, C34.2, C4.-, C5.1, C7.2, C8.-, C9.-, CN1.GND, CN2.GND, D5.A, D6.C, IC1.GND/ADJ, IC2P.V-, IC3.GND, IC4.GND, IC5.GND, IC5.NC, IC5.NC1, IC5.NC2, IC5.NC3, IC5.NC4, IC5.NC5, IC5.NC6, IC5.NC7, IC6.GND, J1-2.S, J2-2.S, J3-2.S, J4-2.S, JP1.6, JP2.GND, JP2.GNDBREAK, R12.1, R15.1, R17.2, R25.1, R26.1, R27.1, R28.1, S1.2, S10.2, S11.2, S12.2, S9.2, U$2.VSS, U$3.VSS, U$4.VSS, U$5.VSS, U1.GND@15, U1.GND@23, U1.GND@35, U1.GND@43, U1.UGND, U3.GND1, U3.GND2
- net HC-05RX: now also R11.2, U2.RX; no longer R14.2, U3.RX
- net HWB: now also IC1.PE2/!HWB, R9.1; no longer R3.1, U1.PE2/!HWB
- net IO10*: now also IC1.PB6(ADC13), U2.TX; no longer U1.PB6(ADC13), U3.TX
- net IO11*: now also IC1.PB7, R11.1, R13.1; no longer R14.1, R15.2, U1.PB7
- net IO12: now also IC1.PD6(ADC9), IC4.OUT; no longer U$2.OUT, U1.PD6(ADC9)
- net IO13*: now also IC1.PC7, JP3.1, S7.P; no longer J2-1.S, S11.1, U1.PC7
- net IO8: now also IC1.PB4(ADC11), IC6.OUT; no longer U$4.OUT, U1.PB4(ADC11)
- net IO9*: now also IC1.PB5(ADC12), U2.PIO11; no longer U1.PB5(ADC12), U3.PIO11
- net MISO: now also IC1.PB3(MISO), ICSP.1; no longer JP1.1, U1.PB3(MISO)
- net MODE1: now also IC6.SYNC/MODE, S1.5; no longer S7.P, U$4.SYNC/MODE
- net MODE2: now also IC3.SYNC/MODE, S2.5; no longer S8.P, U$5.SYNC/MODE
- net MODE3: now also IC4.SYNC/MODE, S3.5; no longer S5.P, U$2.SYNC/MODE
- net MODE4: now also IC5.SYNC/MODE, S4.5; no longer S6.P, U$3.SYNC/MODE
- net MOSI: now also IC1.PB2(MOSI), ICSP.4; no longer JP1.4, U1.PB2(MOSI)
- net N$1: now also R12.1; no longer R6.1
- net N$147: now also R6.2; no longer R29.2
- net N$2: now also R1.2; no longer R7.1
- net N$3: now also R23.2; no longer R8.1
- net PAD1: now also C18.1, PAD1B.PAD, R18.1; no longer C29.2, PAD1B.RECEIVE, PAD1B.RES, R21.2
- net PAD2: now also C16.1, PAD2B.PAD, R17.1; no longer C31.2, PAD2B.RECEIVE, PAD2B.RES, R22.2
- net PAD3: now also C14.1, PAD3B.PAD, R16.1; no longer C25.2, PAD3B.RECEIVE, PAD3B.RES, R19.2
- net PAD4: now also C12.1, PAD4B.PAD, R15.1; no longer C27.2, PAD4B.RECEIVE, PAD4B.RES, R20.2
- net RD+: now also IC1.D+, R24.2; no longer R9.2, U1.D+
- net RD-: now also IC1.D-, R25.2; no longer R10.2, U1.D-
- net RESET: now also D2.A, IC1.!RESET, ICSP.5, R8.2, RESET.1; no longer D1.A, JP1.5, R1.1, S1.1, U1.!RESET
- net RXLED: now also IC1.PB0(SS); no longer U1.PB0(SS)
- net SCK: now also IC1.PB1(SCK), ICSP.3; no longer JP1.3, U1.PB1(SCK)
- net SNS1: now also C19.2, IC6.SNS; no longer C28.1, U$4.SNS
- net SNS2: now also C13.2, IC3.SNS; no longer C30.1, U$5.SNS
- net SNS3: now also C15.2, IC4.SNS; no longer C24.1, U$2.SNS
- net SNS4: now also C17.2, IC5.SNS; no longer C26.1, U$3.SNS
- net SNSK1: now also C19.1, IC6.SNSK, R18.2; no longer C28.2, R21.1, U$4.SNSK
- net SNSK2: now also C13.1, IC3.SNSK, R15.2; no longer C30.2, R22.1, U$5.SNSK
- net SNSK3: now also C15.1, IC4.SNSK, R16.2; no longer C24.2, R19.1, U$2.SNSK
- net SNSK4: now also C17.1, IC5.SNSK, R17.2; no longer C26.2, R20.1, U$3.SNSK
- net STATE: now also R7.1, U2.PIO8; no longer R13.1, U3.PIO8
- net TXLED: now also IC1.PD5; no longer U1.PD5
- net UCAP: now also C3.+, IC1.UCAP; no longer C4.+, U1.UCAP
- net VBAT: now also IC2.VBAT; no longer IC5.VBAT
- net VCC: now also C26.2, C27.+, C28.+; no longer C32.+, C33.+, C34.1
- net VIN: now also +5VDC.PWR, C29.+, D3.C, POWER.VBUS, R21.1, U5.IN; no longer C9.+, CN2.VBUS, D5.C, IC1.IN, JP2.PWR, R11.2
- net VUSB: now also C33.2, C34.+, I1.2, IC1.VBUS; no longer C10.+, C11.2, I1.1, U1.VBUS
- net XTAL1: now also C10.2, IC1.XTAL1, R10.1, Y1.2; no longer C7.1, R2.1, U1.XTAL1, Y1.1
- net XTAL2: now also C9.1, IC1.XTAL2, R10.2, Y1.1; no longer C5.2, R2.2, U1.XTAL2, Y1.2
- net XUSB: now also DATA.VBUS, I1.1; no longer CN1.VBUS, I1.2
